File: KiCad/ESP_Breakout/ESP_Breakout.kicad_sch (KiCad schematic)
At the start: 25 parts, among them J1 Conn_01x15_Socket, J2 Conn_01x15_Socket, J3 Conn_01x03_Pin, J4 Conn_01x03_Pin, J5 Conn_01x03_Pin, J6 Conn_01x03_Pin, J7 Conn_01x15_Socket, J8 Conn_01x15_Socket

Commit message: commit
Parts:
- removed U1: ~, seniorDesign:MODULE_ESP32_DEVKIT_V1, symbol seniorDesign:ESP32_DEVKIT_V1
Connections:
- no-connect marks 30 -> 0
Changed lines of the file:
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@@
 		(color 0 0 0 0)
 	)
-	(no_connect
-		(at 52.07 171.45)
-	)
-	(no_connect
-		(at 52.07 176.53)
-	)
-	(no_connect
-		(at 52.07 189.23)
-	)
-	(no_connect
-		(at 16.51 189.23)
-	)
-	(no_connect
-		(at 52.07 184.15)
-	)
-	(no_connect
-		(at 16.51 191.77)
-	)
-	(no_connect
-		(at 16.51 163.83)
-	)
-	(no_connect
-		(at 16.51 158.75)
-	)
-	(no_connect
-		(at 16.51 186.69)
-	)
-	(no_connect
-		(at 52.07 181.61)
-	)
-	(no_connect
-		(at 52.07 186.69)
-	)
-	(no_connect
-		(at 52.07 173.99)
-	)
-	(no_connect
-		(at 52.07 191.77)
-	)
-	(no_connect
-		(at 16.51 168.91)
-	)
-	(no_connect
-		(at 52.07 158.75)
-	)
-	(no_connect
-		(at 16.51 179.07)
-	)
-	(no_connect
-		(at 16.51 184.15)
-	)
-	(no_connect
-		(at 16.51 166.37)
-	)
-	(no_connect
-		(at 16.51 194.31)
-	)
-	(no_connect
-		(at 16.51 173.99)
-	)
-	(no_connect
-		(at 16.51 181.61)
-	)
-	(no_connect
-		(at 16.51 176.53)
-	)
-	(no_connect
-		(at 16.51 161.29)
-	)
-	(no_connect
-		(at 52.07 168.91)
-	)
-	(no_connect
-		(at 52.07 161.29)
-	)
-	(no_connect
-		(at 52.07 194.31)
-	)
-	(no_connect
-		(at 52.07 163.83)
-	)
-	(no_connect
-		(at 52.07 179.07)
-	)
-	(no_connect
-		(at 52.07 166.37)
-	)
-	(no_connect
-		(at 16.51 171.45)
-	)
 	(wire
 		(pts
@@
 			)
 		)
-		(property "Datasheet" "~"
+		(property "Datasheet" "https://www.digikey.com/en/products/detail/w%C3%BCrth-elektronik/61300311121/4846825"
 			(at 224.79 53.34 0)
 			(effects
@@
 			)
 		)
-		(property "Datasheet" "~"
+		(property "Datasheet" "https://www.digikey.com/en/products/detail/w%C3%BCrth-elektronik/61300311121/4846825"
 			(at 151.13 116.84 0)
 			(effects
@@
 			)
 		)
-		(property "Datasheet" "~"
+		(property "Datasheet" "https://www.digikey.com/en/products/detail/w%C3%BCrth-elektronik/61300311121/4846825"
 			(at 151.13 53.34 0)
 			(effects
@@
 	)
 	(symbol
-		(lib_id "seniorDesign:ESP32_DEVKIT_V1")
-		(at 34.29 176.53 0)
-		(unit 1)
-		(exclude_from_sim no)
-		(in_bom yes)
-		(on_board yes)
-		(dnp no)
-		(fields_autoplaced yes)
-		(property "Reference" "U1"
-			(at 34.29 151.13 0)
-			(effects
-				(font
-					(size 1.27 1.27)
-				)
-			)
-		)
-		(property "Value" "~"
-			(at 34.29 153.67 0)
-			(effects
-				(font
-					(size 1.27 1.27)
-				)
-			)
-		)
-		(property "Footprint" "seniorDesign:MODULE_ESP32_DEVKIT_V1"
-			(at 34.29 176.53 0)
-			(effects
-				(font
-					(size 1.27 1.27)
-				)
-				(hide yes)
-			)
-		)
-		(property "Datasheet" ""
-			(at 34.29 176.53 0)
-			(effects
-				(font
-					(size 1.27 1.27)
-				)
-				(hide yes)
-			)
-		)
-		(property "Description" ""
-			(at 34.29 176.53 0)
-			(effects
-				(font
-					(size 1.27 1.27)
-				)
-				(hide yes)
-			)
-		)
-		(pin "15"
-		)
-		(pin "16"
-		)
-		(pin "17"
-		)
-		(pin ""
-		)
-		(pin "5"
-		)
-		(pin "8"
-		)
-		(pin "10"
-		)
-		(pin "11"
-		)
-		(pin "12"
-		)
-		(pin "13"
-		)
-		(pin "14"
-		)
-		(pin "36"
-		)
-		(pin "39"
-		)
-		(pin "18"
-		)
-		(pin "20"
-		)
-		(pin ""
-		)
-		(pin ""
-		)
-		(pin "41"
-		)
-		(pin "40"
-		)
-		(pin "42"
-		)
-		(pin "38"
-		)
-		(pin "35"
-		)
-		(pin "34"
-		)
-		(pin "27"
-		)
-		(pin "25"
-		)
-		(pin "24"
-		)
-		(pin "22"
-		)
-		(pin "21"
-		)
-		(pin ""
-		)
-		(pin ""
-		)
-		(instances
-			(project ""
-				(path "/dda88b12-46e9-4dfa-bce8-bbcc95317852"
-					(reference "U1")
-					(unit 1)
-				)
-			)
-		)
-	)
-	(symbol
 		(lib_id "B6B-PH-K-S:B6B-PH-K-S")
 		(at 262.89 34.29 0)
@@
 			)
 		)
-		(property "Datasheet" "~"
+		(property "Datasheet" "https://www.digikey.com/en/products/detail/w%C3%BCrth-elektronik/61300311121/4846825"
 			(at 224.79 116.84 0)
 			(effects

Commit message: changed mounting holes
Parts:
- H1, H2, H3, H4: footprint MountingHole:MountingHole_2.5mm -> MountingHole:MountingHole_3.2mm_M3
Changed lines of the file:
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@@
 			)
 		)
-		(property "Footprint" "MountingHole:MountingHole_2.5mm"
+		(property "Footprint" "MountingHole:MountingHole_3.2mm_M3"
 			(at 17.78 24.13 0)
 			(effects
@@
 			)
 		)
-		(property "Footprint" "MountingHole:MountingHole_2.5mm"
+		(property "Footprint" "MountingHole:MountingHole_3.2mm_M3"
 			(at 17.78 36.83 0)
 			(effects
@@
 			)
 		)
-		(property "Footprint" "MountingHole:MountingHole_2.5mm"
+		(property "Footprint" "MountingHole:MountingHole_3.2mm_M3"
 			(at 17.78 17.78 0)
 			(effects
@@
 			)
 		)
-		(property "Footprint" "MountingHole:MountingHole_2.5mm"
+		(property "Footprint" "MountingHole:MountingHole_3.2mm_M3"
 			(at 17.78 30.48 0)
 			(effects
