File: KiCad/Pheonix_Rail/Pheonix_Rail.kicad_sch (KiCad schematic)
At the start: 15 parts, among them J1 1729128, J10 1729128, J11 1729128, J12 1729128, J13 1729128, J2 1729128, J3 1729128, J4 1729128, J5 1729128, J6 1729128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

Commit message: changed mounting holes
Parts:
- H1, H2: footprint MountingHole:MountingHole_2.5mm -> MountingHole:MountingHole_3.2mm_M3
Changed lines of the file:
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@@
 			)
 		)
-		(property "Footprint" "MountingHole:MountingHole_2.5mm"
+		(property "Footprint" "MountingHole:MountingHole_3.2mm_M3"
 			(at 19.05 21.59 0)
 			(effects
@@
 			)
 		)
-		(property "Footprint" "MountingHole:MountingHole_2.5mm"
+		(property "Footprint" "MountingHole:MountingHole_3.2mm_M3"
 			(at 19.05 27.94 0)
 			(effects
