File: KiCad/ESP32_D0WDQ6_bare_metal/ESP32_D0WDQ6_bare_metal.kicad_sch (KiCad schematic)
At the start: 42 parts, among them J2 USB_B_Micro, Q1 SS8050, Q2 SS8050, U1 ESP32-D0WDQ6-V3, U3 W25Q32JVSS, U4 CP2102N-Axx-xQFN28, U5 MIC5365-3.3YD5, X1 40MHz, X2 32kHz768

Commit message: Bare metal update
Added VSPI connector and other stuff
Parts:
- added J1: JST_VSPI_Conn, symbol Connector:Conn_01x04_Pin
- added R10, R11, R12, R13: 22, symbol Device:R
Connections:
- net +3.3V: now also R4.1
- net GND: no longer R4.2
- net XTAL_P: now also R2.2, U1.45 (XTAL_P); no longer C13.1, R2.1, X1.1
- net Chip_En: now reaches C6.1, Q1.3 (C), R1.2, SW_RESET.2, U1.9 (CHIP_PU)
- net 32k768_XN: now reaches C4.1, U1.13 (32K_XN), X2.1
- net at U1.22 (GPIO2): no longer R4.1
- net 32k768_XP: now reaches C19.1, U1.12 (32K_XP), X2.2
- net FLASH_CS: now reaches U1.30 (SD_CMD), U3.1 (~{CS})
- net FLASH_DO: now reaches U1.32 (SD_DATA_0), U3.2 (DO/IO_{1})
- net FLASH_WP: now reaches U1.29 (SD_DATA_3), U3.3 (~{WP}/IO_{2})
- net FLASH_DI: now reaches U1.33 (SD_DATA_1), U3.5 (DI/IO_{0})
- net FLASH_CLK: now reaches U1.31 (SD_CLK), U3.6 (CLK)
- net FLASH_RESET: now reaches U1.28 (SD_DATA_2), U3.7 (~{HOLD}/~{RESET}/IO_{3})
- net at U1.34 (GPIO5): now also R12.1
- net at U1.35 (GPIO18): now also R11.1
- net at U1.36 (GPIO23): now also R13.1
- net at U1.38 (GPIO19): now also R10.1
- new net VSPI_CIPO: J1.1 (Pin_1), R10.2
- new net VSPI_CLK: J1.3 (Pin_3), R11.2
- new net VSPI_COPI: J1.2 (Pin_2), R13.2
- new net VSPI_CS: J1.4 (Pin_4), R12.2, R4.2
- new net XTAL_PIN: C13.1, R2.1, X1.1
