File: KiCad/Stepper_Driver_Board_TI_DRV8434/Stepper_Driver_Board_TI_DRV8434.kicad_pcb (KiCad board)
At the start: 4 copper layers, 0 parts

Commit message: Adding my changes
Parts:
- added C1: 22n, Capacitor_SMD:C_0603_1608Metric_Pad1.08x0.95mm_HandSolder, F.Cu at (157.5, 76.2)
- added C2: 220n, Capacitor_SMD:C_0603_1608Metric_Pad1.08x0.95mm_HandSolder, F.Cu at (147.5, 76.4)
- added C3: 0.01u, Capacitor_SMD:C_0603_1608Metric_Pad1.08x0.95mm_HandSolder, F.Cu at (145.9, 77.7)
- added C4: 0.01u, Capacitor_SMD:C_0603_1608Metric_Pad1.08x0.95mm_HandSolder, F.Cu at (146.5, 83.8)
- added C5: 100u, Capacitor_THT:CP_Radial_D8.0mm_P3.50mm, F.Cu at (199.7, 58.4)
- added C6: 1u, Capacitor_SMD:C_0603_1608Metric_Pad1.08x0.95mm_HandSolder, F.Cu at (157.5, 88.9)
- added C7: 0.1u, Capacitor_SMD:C_0603_1608Metric_Pad1.08x0.95mm_HandSolder, F.Cu at (132.6, 83.7)
- added J1: Motor Connect, Connector_Phoenix_MSTB:PhoenixContact_MSTBA_2,5_4-G-5,08_1x04_P5.08mm_Horizontal, F.Cu at (92.7, 73.7)
- added J2: PWR & DATA Connect, Connector_Phoenix_MSTB:PhoenixContact_MSTBA_2,5_5-G-5,08_1x05_P5.08mm_Horizontal, F.Cu at (188.0, 41.9)
- added R1: 10k, Resistor_SMD:R_0603_1608Metric_Pad0.98x0.95mm_HandSolder, F.Cu at (160.0, 86.4)
- added R2: 10k, Resistor_SMD:R_0603_1608Metric_Pad0.98x0.95mm_HandSolder, F.Cu at (165.1, 86.4)
- added R3: 10k, Resistor_SMD:R_0603_1608Metric_Pad0.98x0.95mm_HandSolder, F.Cu at (165.1, 81.3)
- added R4: 220E, Resistor_SMD:R_0603_1608Metric_Pad0.98x0.95mm_HandSolder, F.Cu at (132.1, 101.6)
- added R5: 4k7, Resistor_SMD:R_0603_1608Metric_Pad0.98x0.95mm_HandSolder, F.Cu at (171.8, 81.3)
- added R6: 220E, Resistor_SMD:R_0603_1608Metric_Pad0.98x0.95mm_HandSolder, F.Cu at (141.3, 91.4)
- added R7: 4k7, Resistor_SMD:R_0603_1608Metric_Pad0.98x0.95mm_HandSolder, F.Cu at (136.4, 96.6)
- added R8: 220E, Resistor_SMD:R_0603_1608Metric_Pad0.98x0.95mm_HandSolder, F.Cu at (136.4, 99.1)
- added R9: 4k7, Resistor_SMD:R_0603_1608Metric_Pad0.98x0.95mm_HandSolder, F.Cu at (136.4, 101.6)
- added SW1: SW_SPDT_MSM, Button_Switch_THT:SW_Slide_SPDT_Straight_CK_OS102011MS2Q, F.Cu at (191.6, 104.1)
- added SW2: SW_SPDT_MSM, Button_Switch_THT:SW_Slide_SPDT_Straight_CK_OS102011MS2Q, F.Cu at (191.6, 116.8)
- added U1: DRV8434PWPR, DRV8434PWPR:TSSOP_34PWPR_TEX, F.Cu at (152.4, 81.3)
- added U2: PC817, Package_DIP:DIP-4_W7.62mm, F.Cu at (184.2, 74.9)
- added U4: 6N137, Package_DIP:DIP-8_W7.62mm, F.Cu at (163.8, 102.9)
- added U6: PC817, Package_DIP:DIP-4_W7.62mm, F.Cu at (185.4, 88.9)

Commit message: worked on layout
Parts:
- added J3: Battery Connect, Connector_Phoenix_MSTB:PhoenixContact_MSTBA_2,5_2-G-5,08_1x02_P5.08mm_Horizontal, F.Cu at (187.2, 87.5)
- U4: moved to B.Cu
- moved SW2 69.3 mm to (152.0, 60.0)
- moved SW1 65.5 mm to (152.0, 52.0)
- moved R4 58.4 mm to (170.9, 58.0)
- moved C5 56.9 mm to (143.0, 63.7), turned to 90 degrees
- moved R9 52.1 mm to (165.0, 58.0), turned to -90 degrees
- moved R6 51.0 mm to (171.0, 50.0)
- moved R8 48.4 mm to (179.0, 76.0), turned to 90 degrees
- moved J1 37.3 mm to (129.8, 69.9)
- moved U4 35.7 mm to (175.8, 69.2), turned to 180 degrees
- moved U6 35.3 mm to (174.8, 55.3), turned to 180 degrees
- moved R7 35.3 mm to (163.0, 73.4), turned to 90 degrees
- moved C7 34.4 mm to (165.0, 72.0), turned to -90 degrees
- moved J2 32.2 mm to (187.2, 74.2), turned to 90 degrees
- moved R5 16.7 mm to (165.0, 66.0), turned to -90 degrees
- moved U2 14.9 mm to (174.8, 63.3), turned to 180 degrees
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Connections:
- J1 pad 3: /BOUT1 -> /BOUT2
- J1 pad 4: /BOUT2 -> /BOUT1
- U1 pad 10: /BOUT2 -> /BOUT1
- U1 pad 11: /BOUT2 -> /BOUT1
- U1 pad 8: /BOUT1 -> /BOUT2
- U1 pad 9: /BOUT1 -> /BOUT2

Commit message: Finished Rough Layout!
Parts:
- U4: moved to F.Cu
- moved SW1 46.1 mm to (175.0, 92.0)
- moved J3 44.3 mm to (143.0, 87.2), turned to 0 degrees
- moved SW2 33.5 mm to (161.0, 92.3)
- moved J2 13.0 mm to (186.2, 87.2)
- moved U4 10.3 mm to (175.8, 79.5)
- moved J1 4.76 mm to (134.3, 68.4)
- moved R4 4.15 mm to (172.0, 62.0)
- moved U2 4.12 mm to (175.8, 67.3)
- moved R6 4.12 mm to (172.0, 54.0)
- moved U6 4.12 mm to (175.8, 59.3)
- moved R3 3.39 mm to (159.8, 79.2), turned to 90 degrees
- moved C6 2.94 mm to (152.0, 81.5), turned to 180 degrees
- moved C5 2.44 mm to (145.2, 62.5), turned to 180 degrees
- moved R9 2.30 mm to (165.5, 60.2)
- moved R5 2.06 mm to (165.5, 68.0)
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Connections:
- J2 pad 3: /ENA_ESP -> /PUL_ESP
- J2 pad 5: /PUL_ESP -> /ENA_ESP
Routing:
- net /M1: track 0.00 -> 33.4 mm
- net /ENA: track 0.00 -> 24.6 mm
- net /M0: track 0.00 -> 24.1 mm
- net GND: track 0.00 -> 18.2 mm, vias 0 -> 9
- net /DIR: track 0.00 -> 17.9 mm
- net /PUL: track 0.00 -> 16.6 mm
- net /ENA_ESP: track 0.00 -> 15.3 mm
- net /DIR_ESP: track 0.00 -> 12.3 mm
- net /PUL_ESP: track 0.00 -> 10.4 mm
- net /VREF: track 0.00 -> 6.97 mm
- net +BATT: track 0.00 -> 5.46 mm, vias 0 -> 3
- net /CPH: track 0.00 -> 4.12 mm
- net /CPL: track 0.00 -> 3.10 mm
- net Net-(U4-C): track 0.00 -> 2.73 mm
- net /FAULT: track 0.00 -> 2.26 mm
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- added copper zone on F.Cu, net +5V
- added copper zone on In2.Cu, net +5V
- added copper zone on F.Cu, net +BATT
- added copper zone on In2.Cu, net +BATT
- added copper zone on F.Cu, net /AOUT1
- added copper zone on F.Cu, net /AOUT2
- added copper zone on F.Cu, net /BOUT1
- added copper zone on F.Cu, net /BOUT2
- added copper zone on B.Cu, net GND
- added copper zone on In1.Cu, net GND
Other:
- board outline added: 75 x 46.8 mm

Commit message: Fixed some via stuff
Routing:
- net Net-(R6-Pad2): track 0.00 -> 5.30 mm
- net Net-(R4-Pad2): track 0.00 -> 5.30 mm
- net +5V: track 1.58 -> 5.84 mm, vias 7 -> 11
- net GND: vias 9 -> 17
Changed lines of the file:
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@@
 		(tags "switch SPDT")
 		(property "Reference" "SW1"
-			(at -4 0 90)
+			(at 4 -3.25 180)
 			(layer "F.SilkS")
 			(effects
@@
 		(tags "phoenix_contact connector MSTBA_01x05_G_5.08mm")
 		(property "Reference" "J2"
-			(at -4.34 3.7775 180)
+			(at -4.59 3.7775 180)
 			(layer "F.SilkS")
 			(effects
@@
 		(tags "resistor handsolder")
 		(property "Reference" "R8"
-			(at 0 2 90)
+			(at 0 1.75 180)
 			(layer "F.SilkS")
 			(effects
@@
 		(tags "capacitor handsolder")
 		(property "Reference" "C1"
-			(at 0 -1.43 90)
+			(at -2.7 -0.1 180)
 			(layer "F.SilkS")
 			(effects
@@
 		(tags "resistor handsolder")
 		(property "Reference" "R7"
-			(at 0 -1.43 90)
+			(at 2.25 -1.5 180)
 			(layer "F.SilkS")
 			(effects
@@
 		(tags "capacitor handsolder")
 		(property "Reference" "C6"
-			(at 2.4 0.3 90)
+			(at 0.25 -1.5 180)
 			(layer "F.SilkS")
 			(effects
@@
 		(tags "phoenix_contact connector MSTBA_01x04_G_5.08mm")
 		(property "Reference" "J1"
-			(at 19.62 4.2775 180)
+			(at 19.87 4.2775 180)
 			(layer "F.SilkS")
 			(effects
@@
 		(tags "capacitor handsolder")
 		(property "Reference" "C4"
-			(at 1 1.25 90)
+			(at -2.6 0 180)
 			(layer "F.SilkS")
 			(effects
@@
 		(tags "capacitor handsolder")
 		(property "Reference" "C7"
-			(at 3 0 90)
+			(at -2.1125 1.5 180)
 			(layer "F.SilkS")
 			(effects
@@
 		(tags "resistor handsolder")
 		(property "Reference" "R5"
-			(at -1 1.5 90)
+			(at -2.5 0 180)
 			(layer "F.SilkS")
 			(effects
@@
 		(tags "capacitor handsolder")
 		(property "Reference" "C3"
-			(at -0.2 1.4 90)
+			(at -0.2 2.5 180)
 			(layer "F.SilkS")
 			(effects
@@
 		(tags "switch SPDT")
 		(property "Reference" "SW2"
-			(at -4.1 0 90)
+			(at 4.5 -3.2975 180)
 			(layer "F.SilkS")
 			(effects
@@
 		(tags "THT DIP DIL PDIP 2.54mm 7.62mm 300mil")
 		(property "Reference" "U4"
-			(at 3.8 10.3 0)
-			(layer "B.SilkS")
+			(at 3.55 -2.25 0)
+			(layer "F.SilkS")
 			(effects
 				(font
@@
 					(thickness 0.15)
 				)
-				(justify mirror)
 			)
 		)
@@
 		(start 181.48125 74.5)
 		(end 180.34375 74.5)
-		(width 0.75)
+		(width 0.5)
 		(layer "F.Cu")
 		(net 5)
@@
 	)
 	(segment
+		(start 145.362563 77.924937)
+		(end 144.75 78.5375)
+		(width 0.3)
+		(layer "F.Cu")
+		(net 5)
+	)
+	(segment
 		(start 150.324993 75.324993)
 		(end 150 75)
@@
 	)
 	(segment
+		(start 147.04725 77.924937)
+		(end 145.362563 77.924937)
+		(width 0.3)
+		(layer "F.Cu")
+		(net 5)
+	)
+	(segment
 		(start 144.6875 72)
 		(end 144.75 72.0625)
@@
 		(start 143.6 72)
 		(end 144.6875 72)
-		(width 0.75)
+		(width 0.5)
 		(layer "F.Cu")
 		(net 5)
@@
 		(start 150 81.5)
 		(end 151.1375 81.5)
-		(width 0.75)
+		(width 0.5)
 		(layer "F.Cu")
 		(net 5)
@@
 		(start 143.68125 78.5)
 		(end 144.81875 78.5)
-		(width 0.75)
-		(layer "F.Cu")
-		(net 5)
-	)
-	(segment
-		(start 147.04725 77.924937)
-		(end 145.362563 77.924937)
-		(width 0.3)
+		(width 0.5)
 		(layer "F.Cu")
 		(net 5)
@@
 		(start 169.93125 62)
 		(end 171.06875 62)
-		(width 0.75)
+		(width 0.5)
 		(layer "F.Cu")
 		(net 5)
@@
 		(start 164.93125 74.25)
 		(end 166.06875 74.25)
-		(width 0.75)
+		(width 0.5)
 		(layer "F.Cu")
 		(net 5)
@@
 		(start 159.75 81.31875)
 		(end 159.75 80.18125)
-		(width 0.75)
+		(width 0.5)
 		(layer "F.Cu")
 		(net 5)
@@
 		(net 5)
 	)
-	(segment
-		(start 145.362563 77.924937)
-		(end 144.75 78.5375)
-		(width 0.3)
-		(layer "F.Cu")
+	(via
+		(at 150 74)
+		(size 0.7)
+		(drill 0.3)
+		(layers "F.Cu" "B.Cu")
+		(free yes)
+		(net 5)
+	)
+	(via
+		(at 151.2 75)
+		(size 0.7)
+		(drill 0.3)
+		(layers "F.Cu" "B.Cu")
+		(free yes)
 		(net 5)
 	)
@@
 	)
 	(via
+		(at 150 75.9)
+		(size 0.7)
+		(drill 0.3)
+		(layers "F.Cu" "B.Cu")
+		(free yes)
+		(net 5)
+	)
+	(via
 		(at 143.6 72)
 		(size 0.7)
@@
 	)
 	(via
+		(at 151.1 73.4)
+		(size 0.7)
+		(drill 0.3)
+		(layers "F.Cu" "B.Cu")
+		(free yes)
+		(net 5)
+	)
+	(via
+		(at 151.1 76.6)
+		(size 0.7)
+		(drill 0.3)
+		(layers "F.Cu" "B.Cu")
+		(free yes)
+		(net 5)
+	)
+	(via
 		(at 169.93125 54)
 		(size 0.7)
@@
 	)
 	(via
+		(at 148.8 75)
+		(size 0.7)
+		(drill 0.3)
+		(layers "F.Cu" "B.Cu")
+		(free yes)
+		(net 5)
+	)
+	(via
 		(at 150 81.5)
 		(size 0.7)
@@
 	)
 	(via
+		(at 148.9 76.6)
+		(size 0.7)
+		(drill 0.3)
+		(layers "F.Cu" "B.Cu")
+		(free yes)
+		(net 5)
+	)
+	(via
 		(at 181.48125 74.5)
 		(size 0.7)
@@
 	)
 	(via
+		(at 148.9 73.4)
+		(size 0.7)
+		(drill 0.3)
+		(layers "F.Cu" "B.Cu")
+		(free yes)
+		(net 5)
+	)
+	(via
 		(at 143.68125 78.5)
 		(size 0.7)
@@
 	)
 	(segment
+		(start 165.5 62.25)
+		(end 165.5 61.1625)
+		(width 0.5)
+		(layer "F.Cu")
+		(net 6)
+	)
+	(segment
+		(start 163.5 74.0875)
+		(end 163.5 73)
+		(width 0.5)
+		(layer "F.Cu")
+		(net 6)
+	)
+	(segment
+		(start 165.5 68.9125)
+		(end 165.5 70)
+		(width 0.5)
+		(layer "F.Cu")
+		(net 6)
+	)
+	(segment
+		(start 166 72.5)
+		(end 165 72.5)
+		(width 0.5)
+		(layer "F.Cu")
+		(net 6)
+	)
+	(segment
 		(start 154.174937 72.075063)
 		(end 154.25 72)
@@
 	)
 	(via
+		(at 165 72.5)
+		(size 0.6)
+		(drill 0.3)
+		(layers "F.Cu" "B.Cu")
+		(free yes)
+		(net 6)
+	)
+	(via
 		(at 154 81.5)
 		(size 0.6)
@@
 	)
 	(via
+		(at 165.5 62.25)
+		(size 0.6)
+		(drill 0.3)
+		(layers "F.Cu" "B.Cu")
+		(free yes)
+		(net 6)
+	)
+	(via
 		(at 156.5875 80.25)
 		(size 0.6)
@@
 	)
 	(via
+		(at 163.5 73)
+		(size 0.6)
+		(drill 0.3)
+		(layers "F.Cu" "B.Cu")
+		(free yes)
+		(net 6)
+	)
+	(via
 		(at 153.75 80.25)
 		(size 0.6)
@@
 	)
 	(via
-		(at 154.4 76)
+		(at 165.5 70)
+		(size 0.6)
+		(drill 0.3)
+		(layers "F.Cu" "B.Cu")
+		(free yes)
+		(net 6)
+	)
+	(via
+		(at 154.5 75.75)
 		(size 0.6)
 		(drill 0.3)
@@
 	)
 	(via
-		(at 154.4 76.6)
+		(at 154.75 76.624951)
 		(size 0.6)
 		(drill 0.3)
@@
 	)
 	(segment
+		(start 175.75 62.75)
+		(end 175.8 62.8)
+		(width 0.5)
+		(layer "F.Cu")
+		(net 16)
+	)
+	(segment
+		(start 175.8 62.8)
+		(end 175.8 64.735)
+		(width 0.5)
+		(layer "F.Cu")
+		(net 16)
+	)
+	(segment
+		(start 175.25 62)
+		(end 175.75 62.5)
+		(width 0.5)
+		(layer "F.Cu")
+		(net 16)
+	)
+	(segment
+		(start 175.75 62.5)
+		(end 175.75 62.75)
+		(width 0.5)
+		(layer "F.Cu")
+		(net 16)
+	)
+	(segment
+		(start 172.9125 62)
+		(end 175.25 62)
+		(width 0.5)
+		(layer "F.Cu")
+		(net 16)
+	)
+	(segment
 		(start 158.124965 73.375035)
 		(end 164.4125 67.0875)
@@
 	)
 	(segment
+		(start 175.25 54)
+		(end 175.8 54.55)
+		(width 0.5)
+		(layer "F.Cu")
+		(net 18)
+	)
+	(segment
+		(start 172.9125 54)
+		(end 175.25 54)
+		(width 0.5)
+		(layer "F.Cu")
+		(net 18)
+	)
+	(segment
+		(start 175.8 54.55)
+		(end 175.8 56.735)
+		(width 0.5)
+		(layer "F.Cu")
+		(net 18)
+	)
+	(segment
 		(start 161 74)
 		(end 160.974979 74.025021)
@@
 		(polygon
 			(pts
-				(xy 152.25 75.8) (xy 154 75.8) (xy 154.2 75.65) (xy 154.75 75.65) (xy 154.75 76.95) (xy 154.2 76.95)
-				(xy 154 76.8) (xy 152.25 76.8)
+				(xy 152.25 75.8) (xy 154 75.8) (xy 154.3 75.4) (xy 154.825001 75.3625) (xy 155.011296 75.525081)
+				(xy 155.085492 76.675121) (xy 154.875 76.9125) (xy 154.2 76.95) (xy 154 76.8) (xy 152.25 76.8)
 			)
 		)

Commit message: driver board updating
Routing:
- added copper zone on F.Cu, net GND
Other:
- board text added: "1 Z 0"
- board text added: "M0:"
- board text added: "M0=0, M1=1 -> 1/4 M0=1, M1=1 -> 1/8 M0=Z, M1=1 -> 1/6"
- board text added: "M1:"
Changed lines of the file:
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@@
 		)
 		(pad_to_mask_clearance 0)
-		(solder_mask_min_width 0.125)
 		(allow_soldermask_bridges_in_footprints no)
 		(tenting front back)
@@
 			(outputformat 1)
 			(mirror no)
-			(drillshape 1)
+			(drillshape 0)
 			(scaleselection 1)
-			(outputdirectory "")
+			(outputdirectory "/Users/phennessey/Desktop/")
 		)
 	)
@@
 				(type solid)
 			)
-			(layer "B.CrtYd")
+			(layer "F.CrtYd")
 		)
 		(fp_line
@@
 				(type solid)
 			)
-			(layer "B.CrtYd")
+			(layer "F.CrtYd")
 		)
 		(fp_line
@@
 				(type solid)
 			)
-			(layer "B.CrtYd")
+			(layer "F.CrtYd")
 		)
 		(fp_line
@@
 				(type solid)
 			)
-			(layer "B.CrtYd")
+			(layer "F.CrtYd")
 		)
 		(fp_line
@@
 		)
 		(embedded_fonts no)
-		(model "${KICAD8_3DMODEL_DIR}/Button_Switch_THT.3dshapes/SW_Slide_SPDT_Straight_CK_OS102011MS2Q.wrl"
+		(model "${KICAD9_3DMODEL_DIR}/Button_Switch_THT.3dshapes/SW_Slide_SPDT_Straight_CK_OS102011MS2Q.step"
 			(offset
 				(xyz 0 0 0)
@@
 				(type solid)
 			)
-			(layer "B.CrtYd")
+			(layer "F.CrtYd")
 		)
 		(fp_line
@@
 				(type solid)
 			)
-			(layer "B.CrtYd")
+			(layer "F.CrtYd")
 		)
 		(fp_line
@@
 				(type solid)
 			)
-			(layer "B.CrtYd")
+			(layer "F.CrtYd")
 		)
 		(fp_line
@@
 				(type solid)
 			)
-			(layer "B.CrtYd")
+			(layer "F.CrtYd")
 		)
 		(fp_line
@@
 		)
 		(embedded_fonts no)
-		(model "${KICAD8_3DMODEL_DIR}/Button_Switch_THT.3dshapes/SW_Slide_SPDT_Straight_CK_OS102011MS2Q.wrl"
+		(model "${KICAD9_3DMODEL_DIR}/Button_Switch_THT.3dshapes/SW_Slide_SPDT_Straight_CK_OS102011MS2Q.step"
 			(offset
 				(xyz 0 0 0)
@@
 		(layer "Edge.Cuts")
 	)
+	(gr_text "M0=0, M1=1 -> 1/4\nM0=1, M1=1 -> 1/8\nM0=Z, M1=1 -> 1/6"
+		(at 183.4 96.7 0)
+		(layer "F.SilkS")
+		(effects
+			(font
+				(size 0.75 0.75)
+				(thickness 0.1)
+			)
+			(justify left bottom)
+		)
+	)
+	(gr_text "M0:\n"
+		(at 157.9 96.4 0)
+		(layer "F.SilkS")
+		(effects
+			(font
+				(size 1 1)
+				(thickness 0.1)
+			)
+			(justify left bottom)
+		)
+	)
+	(gr_text "1 Z 0\n"
+		(at 174.8 96.1 0)
+		(layer "F.SilkS")
+		(effects
+			(font
+				(size 1 1)
+				(thickness 0.2)
+				(bold yes)
+			)
+			(justify left bottom)
+		)
+	)
+	(gr_text "M1:"
+		(at 171.9 96.1 0)
+		(layer "F.SilkS")
+		(effects
+			(font
+				(size 1 1)
+				(thickness 0.1)
+			)
+			(justify left bottom)
+		)
+	)
+	(gr_text "1 Z 0\n"
+		(at 160.9 96.4 0)
+		(layer "F.SilkS")
+		(effects
+			(font
+				(size 1 1)
+				(thickness 0.2)
+				(bold yes)
+			)
+			(justify left bottom)
+		)
+	)
 	(segment
 		(start 152.95275 69.79725)
@@
 	)
 	(segment
-		(start 160.75 77.25)
-		(end 160.725049 77.274951)
-		(width 0.3)
-		(layer "F.Cu")
-		(net 23)
-	)
-	(segment
 		(start 163 92.2975)
 		(end 163 80.5)
@@
 	(segment
 		(start 163 80.5)
-		(end 161.25 78.75)
+		(end 163.1 80.4)
 		(width 0.3)
 		(layer "F.Cu")
@@
 	)
 	(segment
-		(start 161.25 77.25)
-		(end 160.75 77.25)
+		(start 163.1 80.4)
+		(end 163.1 79.1)
 		(width 0.3)
 		(layer "F.Cu")
@@
 	)
 	(segment
-		(start 160.725049 77.274951)
-		(end 152.95275 77.274951)
+		(start 163.1 79.1)
+		(end 161.274951 77.274951)
 		(width 0.3)
 		(layer "F.Cu")
@@
 	)
 	(segment
-		(start 161.25 78.75)
-		(end 161.25 77.25)
+		(start 161.274951 77.274951)
+		(end 152.95275 77.274951)
 		(width 0.3)
 		(layer "F.Cu")
@@
 			)
 		)
+	)
+	(zone
+		(net 5)
+		(net_name "GND")
+		(layer "F.Cu")
+		(hatch edge 0.5)
+		(priority 10)
+		(connect_pads yes
+			(clearance 0.3)
+		)
+		(min_thickness 0.25)
+		(filled_areas_thickness no)
+		(fill yes
+			(thermal_gap 0.5)
+			(thermal_bridge_width 0.5)
+		)
+		(polygon
+			(pts
+				(xy 148 70) (xy 148 80) (xy 152 80) (xy 152 70)
+			)
+		)
