File: KiCad/2ESP_Breakout/2ESP_Breakout.kicad_pcb (KiCad board)
At the start: 2 copper layers, 132.1 x 101.6 mm, 36 parts, among them J1 Conn_01x02_Socket, J10 Conn_01x02_Socket, J11 Conn_01x02_Socket, J12 Conn_01x02_Socket, J13 Conn_01x02_Socket, J14 Conn_01x02_Socket, J15 Conn_01x02_Socket, J16 Conn_01x02_Socket, J2 Conn_01x02_Socket, J3 Conn_01x02_Socket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

Commit message: Cleaned up routing
Parts:
- added Buck_Header1: Conn_01x04_Pin, Connector_PinHeader_2.54mm:PinHeader_1x04_P2.54mm_Vertical, F.Cu at (218.4, 114.3)
- added H1: MountingHole, MountingHole:MountingHole_3.2mm_M3, F.Cu at (223.0, 67.3)
- added H2: MountingHole, MountingHole:MountingHole_3.2mm_M3, F.Cu at (102.9, 130.6)
- added H3: MountingHole, MountingHole:MountingHole_3.2mm_M3, F.Cu at (102.9, 67.3)
- added H4: MountingHole, MountingHole:MountingHole_3.2mm_M3, F.Cu at (223.0, 130.6)
- moved LIFT2 96.7 mm to (205.7, 73.7), turned to -90 degrees
- moved LIFT1 91.6 mm to (213.4, 73.7), turned to -90 degrees
- moved J5 77.6 mm to (127.0, 78.7), turned to 180 degrees
- moved J4 70.4 mm to (127.0, 72.4), turned to 180 degrees
- moved J3 63.5 mm to (127.0, 66.0), turned to 180 degrees
- moved TURN4 33.9 mm to (114.3, 158.8)
- moved LIFT3 10.2 mm to (205.7, 90.3)
- moved LIFT4 10.2 mm to (213.4, 90.3)
- moved DRIVE2 5.08 mm to (114.3, 109.2)
- moved DRIVE4 5.08 mm to (114.3, 94.0)
- moved J10 2.54 mm to (189.2, 132.1)
- moved J15 2.54 mm to (196.8, 149.9)
- moved ESP2L_1 2.54 mm to (147.3, 121.9)
- moved ESP2L_2 2.54 mm to (137.2, 121.9)
- moved ESP2R_1 2.54 mm to (172.7, 121.9)
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Connections:
- ESP1L_1 pad 15: Net-(ESP1L_1-VIN) -> Net-(Buck_Header1-Pin_4)
- ESP1L_1 pad 6: /LIFT2_PULSE -> /Limit_1_32
- ESP1L_1 pad 7: /LIFT1_PULSE -> /Limit_1_33
- ESP1L_1 pad 8: /LIFT_ENABLE -> /Limit_1_25
- ESP1L_2 pad 15: Net-(ESP1L_1-VIN) -> Net-(Buck_Header1-Pin_4)
- ESP1L_2 pad 6: /LIFT2_PULSE -> /Limit_1_32
- ESP1L_2 pad 7: /LIFT1_PULSE -> /Limit_1_33
- ESP1L_2 pad 8: /LIFT_ENABLE -> /Limit_1_25
- ESP1R_1 pad 5: /Limit_1_21 -> /LIFT2_PULSE
- ESP1R_1 pad 6: /Limit_1_19 -> /LIFT1_PULSE
- ESP1R_1 pad 7: /Limit_1_18 -> /LIFT_ENABLE
- ESP1R_2 pad 5: /Limit_1_21 -> /LIFT2_PULSE
- ESP1R_2 pad 6: /Limit_1_19 -> /LIFT1_PULSE
- ESP1R_2 pad 7: /Limit_1_18 -> /LIFT_ENABLE
- ESP2L_1 pad 10: /TURN2_DIRECTION -> /TURN4_DIRECTION
- ESP2L_1 pad 15: Net-(ESP2L_1-VIN) -> Net-(Buck_Header1-Pin_4)
- ESP2L_1 pad 6: /TURN4_PULSE -> /TURN3_PULSE
- ESP2L_1 pad 7: /TURN4_DIRECTION -> /TURN2_PULSE
- ESP2L_1 pad 8: /TURN3_PULSE -> /TURN2_DIRECTION
- ESP2L_1 pad 9: /TURN2_PULSE -> /TURN4_PULSE
- ESP2L_2 pad 10: /TURN2_DIRECTION -> /TURN4_DIRECTION
- ESP2L_2 pad 15: Net-(ESP2L_1-VIN) -> Net-(Buck_Header1-Pin_4)
- ESP2L_2 pad 6: /TURN4_PULSE -> /TURN3_PULSE
- ESP2L_2 pad 7: /TURN4_DIRECTION -> /TURN2_PULSE
- ESP2L_2 pad 8: /TURN3_PULSE -> /TURN2_DIRECTION
- ESP2L_2 pad 9: /TURN2_PULSE -> /TURN4_PULSE
- J3 pad 1: /Limit_1_21 -> /Limit_1_32
- J4 pad 1: /Limit_1_19 -> /Limit_1_33
- J5 pad 1: /Limit_1_18 -> /Limit_1_25
Routing:
- net Net-(Buck_Header1-Pin_4): track 0.00 -> 217.7 mm
- net /LIFT_DIRECTION: track 187.1 -> 111.7 mm
- net /LIFT_ENABLE: track 148.5 -> 74.8 mm
- net /Limit_1_32: track 0.00 -> 32.6 mm
- net /Limit_1_18: track 31.8 -> 0.00 mm
- net /TURN_ENABLE: track 33.6 -> 64.7 mm
- net /Limit_1_33: track 0.00 -> 28.8 mm
- net /Limit_1_25: track 0.00 -> 26.1 mm
- net /Limit_1_19: track 24.1 -> 0.00 mm
- net /LIFT2_PULSE: track 52.3 -> 35.1 mm
- net /Limit_1_21: track 16.5 -> 0.00 mm
- net /LIFT4_PULSE: track 54.0 -> 43.3 mm
- net Net-(ESP2L_1-VIN): track 10.2 -> 0.00 mm
- net Net-(ESP1L_1-VIN): track 10.2 -> 0.00 mm
- net /DRIVE_ENABLE: track 74.9 -> 64.7 mm
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- added copper zone on F.Cu, net GND
Other:
- board text added: "MountingHole"
- board text added: "Neon Carrot Motor Control Board V2"

Commit message: Needs some more work on 2esp
Parts:
- removed J1, J8: Conn_01x02_Socket, Connector_JST:JST_PH_B2B-PH-K_1x02_P2.00mm_Vertical
- added ESP3L1: Conn_01x15_Socket, Connector_PinSocket_2.54mm:PinSocket_1x15_P2.54mm_Vertical, F.Cu at (224.8, 110.5)
- added ESP3R1: Conn_01x15_Socket, Connector_PinSocket_2.54mm:PinSocket_1x15_P2.54mm_Vertical, F.Cu at (224.8, 135.9)
- moved Buck_Header1 120.8 mm to (97.8, 119.4), turned to 0 degrees
- moved H2 40.8 mm to (102.9, 171.4)
- moved H4 40.8 mm to (223.0, 171.4)
- moved J12 19.1 mm to (204.5, 156.2)
- moved J13 19.1 mm to (189.2, 158.8)
- moved J14 19.1 mm to (189.2, 166.4)
- moved TURN1 19.1 mm to (121.9, 177.8)
- moved TURN4 19.1 mm to (114.3, 177.8)
- moved ESP2L_1 19.0 mm to (147.3, 141.0)
- moved ESP2L_2 19.0 mm to (137.2, 141.0)
- moved ESP2R_1 19.0 mm to (172.7, 141.0)
- moved ESP2R_2 19.0 mm to (182.9, 141.0)
- moved J9 19.0 mm to (196.8, 143.5)
- moved J10 19.0 mm to (189.2, 151.1)
- moved J11 19.0 mm to (196.8, 153.7)
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Connections:
- ESP1R_1 pad 1: /Limit_1_23 -> /LIFT_DIRECTION
- ESP1R_1 pad 10: Net-(ESP1R_1-RX2) -> /TX_PARENT
- ESP1R_1 pad 9: /LIFT_DIRECTION -> /TX_CHILD1
- ESP1R_2 pad 1: /Limit_1_23 -> /LIFT_DIRECTION
- ESP1R_2 pad 10: Net-(ESP1R_1-RX2) -> /TX_PARENT
- ESP1R_2 pad 9: /LIFT_DIRECTION -> /TX_CHILD1
- ESP2R_1 pad 1: /Limit_2_23 -> /TURN3_DIRECTION
- ESP2R_1 pad 10: Net-(ESP2R_1-RX2) -> /TX_PARENT
- ESP2R_1 pad 9: /TURN3_DIRECTION -> /TX_CHILD2
- ESP2R_2 pad 1: /Limit_2_23 -> /TURN3_DIRECTION
- ESP2R_2 pad 10: Net-(ESP2R_1-RX2) -> /TX_PARENT
- ESP2R_2 pad 9: /TURN3_DIRECTION -> /TX_CHILD2
Routing:
- net /TX_CHILD1: track 0.00 -> 216.4 mm
- net /TX_PARENT: track 0.00 -> 160.8 mm
- net /TX_CHILD2: track 0.00 -> 64.0 mm
- net Net-(Buck_Header1-Pin_4): track 217.7 -> 169.5 mm
- net /TURN3_DIRECTION: track 109.9 -> 91.6 mm
- net /Limit_2_23: track 16.5 -> 0.00 mm
- net /Limit_1_23: track 16.5 -> 0.00 mm
- net Net-(ESP2R_1-RX2): track 10.2 -> 0.00 mm
- net Net-(ESP1R_1-RX2): track 10.2 -> 0.00 mm
- net /Limit_1_22: track 24.1 -> 16.5 mm
- net /BACK_DRIVE_PULSE: track 35.0 -> 42.3 mm
- net /BACK_DRIVE_DIRECTION: track 34.4 -> 41.7 mm
- net /LIFT_DIRECTION: track 111.7 -> 107.2 mm
- net /DRIVE_ENABLE: track 64.7 -> 67.6 mm
- net /FRONT_DRIVE_PULSE: track 35.2 -> 38.1 mm
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- added copper zone on F.Cu, net /LIFT_DIRECTION
Other:
- board size 132.1 x 101.6 mm -> 134.6 x 119.4 mm

Commit message: Final KiCad stuff for 2ESP and Driver Board
Parts:
- removed ESP3L1, ESP3R1: Conn_01x15_Socket, Connector_PinSocket_2.54mm:PinSocket_1x15_P2.54mm_Vertical
- added ESP3L_1: Conn_01x15_Socket, Connector_PinSocket_2.54mm:PinSocket_1x15_P2.54mm_Vertical, F.Cu at (224.8, 110.5)
- added ESP3L_2: Conn_01x15_Socket, Connector_PinSocket_2.54mm:PinSocket_1x15_P2.54mm_Vertical, F.Cu at (224.8, 106.7)
- added ESP3L_3: Conn_01x15_Socket, Connector_PinSocket_2.54mm:PinSocket_1x15_P2.54mm_Vertical, F.Cu at (224.8, 139.7)
- added ESP3R_1: Conn_01x15_Socket, Connector_PinSocket_2.54mm:PinSocket_1x15_P2.54mm_Vertical, F.Cu at (224.8, 135.9)
- moved DRIVE1 2.54 mm to (116.8, 101.4)
- moved DRIVE2 2.54 mm to (109.2, 101.4)
- moved H1 2.54 mm to (223.0, 64.8)
- moved H3 2.54 mm to (102.9, 64.8)
- moved J2 2.54 mm to (189.2, 68.6)
- moved J3 2.54 mm to (127.0, 63.5)
- moved J4 2.54 mm to (127.0, 69.8)
- moved J6 2.54 mm to (189.2, 83.8)
- moved J7 2.54 mm to (189.2, 91.4)
- moved DRIVE3 2.54 mm to (116.8, 86.3)
- moved DRIVE4 2.54 mm to (109.2, 86.2)
- moved ESP1L_1 2.54 mm to (147.3, 66.0)
- moved ESP1L_2 2.54 mm to (137.2, 66.0)
- moved ESP1R_1 2.54 mm to (172.7, 66.0)
- moved ESP1R_2 2.54 mm to (182.9, 66.0)
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Connections:
- net Net-(Buck_Header1-Pin_4) renamed /5V
- ESP1R_1 pad 10: /TX_PARENT -> /TX_PARENT1
- ESP1R_2 pad 10: /TX_PARENT -> /TX_PARENT1
- ESP2R_1 pad 10: /TX_PARENT -> /TX_PARENT2
- ESP2R_2 pad 10: /TX_PARENT -> /TX_PARENT2
Routing:
- net /5V: track 169.5 -> 340.8 mm
- net /TX_PARENT: track 160.8 -> 0.00 mm
- net /TX_PARENT1: track 0.00 -> 98.9 mm
- net /TX_PARENT2: track 0.00 -> 70.8 mm
- net /TX_CHILD1: track 216.4 -> 220.6 mm
- net Net-(ESP3L_3-VP): track 0.00 -> 3.81 mm
- net Net-(ESP3L_3-VN): track 0.00 -> 3.81 mm
- net Net-(ESP3L_3-VIN): track 0.00 -> 3.81 mm
- net Net-(ESP3L_3-EN): track 0.00 -> 3.81 mm
- net Net-(ESP3L_3-D35): track 0.00 -> 3.81 mm
- net Net-(ESP3L_3-D34): track 0.00 -> 3.81 mm
- net Net-(ESP3L_3-D32): track 0.00 -> 3.81 mm
- net Net-(ESP3L_3-D14): track 0.00 -> 3.81 mm
- net Net-(ESP3L_3-D13): track 0.00 -> 3.81 mm
- net Net-(ESP3L_3-D12): track 0.00 -> 3.81 mm
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- added copper zone on F.Cu, net /5V
Other:
- board size 134.6 x 119.4 mm -> 134.6 x 124.5 mm
- board text added: "ESP1"
- board text added: "ESP2"
- board text added: "ESP3"
- board text added: "NEON CARROT MOTOR CONTROL BOARD V2"
- board text removed: "Neon Carrot Motor Control Board V2"
