File: KiCad/12_Driver_Board/12_Driver_Board.kicad_pcb (KiCad board)
At the start: 4 copper layers, 75 x 46.8 mm, 25 parts, among them J1 Motor Connect, J2 PWR & DATA Connect, J3 Battery Connect, SW1 SW_SPDT_MSM, SW2 SW_SPDT_MSM, U1 DRV8434PWPR, U2 PC817, U4 6N137, U6 PC817

Commit message: Adding Cad files
Parts:
- removed U1: DRV8434PWPR, DRV8434PWPR:TSSOP_34PWPR_TEX
- added C10: 0.01u, Capacitor_SMD:C_0603_1608Metric, F.Cu at (440.2, 150.1)
- added C11: 22n, Capacitor_SMD:C_0603_1608Metric, F.Cu at (429.3, 209.6)
- added C12: 1u, Capacitor_SMD:C_0603_1608Metric, F.Cu at (432.6, 198.1)
- added C13: 220n, Capacitor_SMD:C_0603_1608Metric, F.Cu at (438.4, 211.1)
- added C14: 0.01u, Capacitor_SMD:C_0603_1608Metric, F.Cu at (440.2, 208.8)
- added C15: 0.01u, Capacitor_SMD:C_0603_1608Metric, F.Cu at (440.2, 200.9)
- added C16: 22n, Capacitor_SMD:C_0603_1608Metric, F.Cu at (429.3, 260.4)
- added C17: 1u, Capacitor_SMD:C_0603_1608Metric, F.Cu at (432.6, 248.9)
- added C18: 220n, Capacitor_SMD:C_0603_1608Metric, F.Cu at (438.4, 261.9)
- added C19: 0.01u, Capacitor_SMD:C_0603_1608Metric, F.Cu at (440.2, 259.6)
- added C20: 0.01u, Capacitor_SMD:C_0603_1608Metric, F.Cu at (440.2, 251.7)
- added C21: 22n, Capacitor_SMD:C_0603_1608Metric, F.Cu at (160.8, 352.8)
- added C22: 1u, Capacitor_SMD:C_0603_1608Metric, F.Cu at (157.5, 364.0)
- added C23: 220n, Capacitor_SMD:C_0603_1608Metric, F.Cu at (151.6, 351.0)
- added C24: 0.01u, Capacitor_SMD:C_0603_1608Metric, F.Cu at (149.9, 353.3)
- added C25: 0.01u, Capacitor_SMD:C_0603_1608Metric, F.Cu at (149.9, 361.2)
- added C26: 22n, Capacitor_SMD:C_0603_1608Metric, F.Cu at (160.8, 302.0)
- added C27: 1u, Capacitor_SMD:C_0603_1608Metric, F.Cu at (157.5, 313.2)
- added C28: 220n, Capacitor_SMD:C_0603_1608Metric, F.Cu at (151.6, 300.2)
- added C29: 0.01u, Capacitor_SMD:C_0603_1608Metric, F.Cu at (149.9, 302.5)
- added C30: 0.01u, Capacitor_SMD:C_0603_1608Metric, F.Cu at (149.9, 310.4)
- added C31: 22n, Capacitor_SMD:C_0603_1608Metric, F.Cu at (160.8, 98.8)
- added C32: 1u, Capacitor_SMD:C_0603_1608Metric, F.Cu at (157.5, 110.0)
- added C33: 220n, Capacitor_SMD:C_0603_1608Metric, F.Cu at (151.6, 97.0)
- added C34: 0.01u, Capacitor_SMD:C_0603_1608Metric, F.Cu at (149.9, 107.2)
- added C35: 0.01u, Capacitor_SMD:C_0603_1608Metric, F.Cu at (149.9, 99.3)
- added C36: 22n, Capacitor_SMD:C_0603_1608Metric, F.Cu at (160.8, 149.6)
- added C37: 1u, Capacitor_SMD:C_0603_1608Metric, F.Cu at (157.5, 160.8)
- added C38: 220n, Capacitor_SMD:C_0603_1608Metric, F.Cu at (151.6, 147.8)
- added C39: 0.01u, Capacitor_SMD:C_0603_1608Metric, F.Cu at (149.9, 150.1)
- added C40: 0.01u, Capacitor_SMD:C_0603_1608Metric, F.Cu at (149.9, 158.0)
- added C41: 22n, Capacitor_SMD:C_0603_1608Metric, F.Cu at (160.8, 200.4)
- added C42: 1u, Capacitor_SMD:C_0603_1608Metric, F.Cu at (157.5, 211.6)
- added C43: 220n, Capacitor_SMD:C_0603_1608Metric, F.Cu at (151.6, 198.6)
- added C44: 0.01u, Capacitor_SMD:C_0603_1608Metric, F.Cu at (149.9, 200.9)
- added C45: 0.01u, Capacitor_SMD:C_0603_1608Metric, F.Cu at (149.9, 208.8)
- added C46: 22n, Capacitor_SMD:C_0603_1608Metric, F.Cu at (160.8, 251.2)
- added C47: 1u, Capacitor_SMD:C_0603_1608Metric, F.Cu at (157.5, 262.4)
- added C48: 220n, Capacitor_SMD:C_0603_1608Metric, F.Cu at (151.6, 249.4)
- added C49: 0.01u, Capacitor_SMD:C_0603_1608Metric, F.Cu at (149.9, 251.7)
- added C50: 0.01u, Capacitor_SMD:C_0603_1608Metric, F.Cu at (149.9, 259.6)
- added C51: 22n, Capacitor_SMD:C_0603_1608Metric, F.Cu at (429.3, 311.2)
- added C52: 1u, Capacitor_SMD:C_0603_1608Metric, F.Cu at (432.6, 299.7)
- added C53: 220n, Capacitor_SMD:C_0603_1608Metric, F.Cu at (438.4, 312.7)
- added C54: 0.01u, Capacitor_SMD:C_0603_1608Metric, F.Cu at (440.2, 310.4)
- added C55: 0.01u, Capacitor_SMD:C_0603_1608Metric, F.Cu at (440.2, 302.5)
- added C56: 22n, Capacitor_SMD:C_0603_1608Metric, F.Cu at (429.3, 362.0)
- added C57: 1u, Capacitor_SMD:C_0603_1608Metric, F.Cu at (432.6, 350.5)
- added C58: 220n, Capacitor_SMD:C_0603_1608Metric, F.Cu at (438.4, 363.5)
- added C59: 0.01u, Capacitor_SMD:C_0603_1608Metric, F.Cu at (440.2, 361.2)
- added C60: 0.01u, Capacitor_SMD:C_0603_1608Metric, F.Cu at (440.2, 353.3)
- added C61: 0.1u, Capacitor_SMD:C_0603_1608Metric, F.Cu at (389.9, 145.6)
- added C62: 0.1u, Capacitor_SMD:C_0603_1608Metric, F.Cu at (389.9, 94.8)
- added C63: 0.1u, Capacitor_SMD:C_0603_1608Metric, F.Cu at (389.9, 196.4)
- added C64: 0.1u, Capacitor_SMD:C_0603_1608Metric, F.Cu at (389.9, 247.2)
- added C65: 0.1u, Capacitor_SMD:C_0603_1608Metric, F.Cu at (199.4, 133.8)
- added C66: 0.1u, Capacitor_SMD:C_0603_1608Metric, F.Cu at (199.4, 235.4)
- added C67: 0.1u, Capacitor_SMD:C_0603_1608Metric, F.Cu at (199.4, 359.9)
- added C68: 0.1u, Capacitor_SMD:C_0603_1608Metric, F.Cu at (389.9, 298.0)
- added C69: 0.1u, Capacitor_SMD:C_0603_1608Metric, F.Cu at (389.9, 348.8)
- added C70: 0.1u, Capacitor_SMD:C_0603_1608Metric, F.Cu at (199.4, 309.1)
- added C8: 220n, Capacitor_SMD:C_0603_1608Metric, F.Cu at (438.4, 160.3)
- added C9: 0.01u, Capacitor_SMD:C_0603_1608Metric, F.Cu at (440.2, 158.0)
- added ESP1L_1: Conn_01x15_Socket, Connector_PinSocket_2.54mm:PinSocket_1x15_P2.54mm_Vertical, F.Cu at (279.4, 144.8)
- added ESP1R_1: Conn_01x15_Socket, Connector_PinSocket_2.54mm:PinSocket_1x15_P2.54mm_Vertical, F.Cu at (304.8, 144.8)
- added ESP2L_1: Conn_01x15_Socket, Connector_PinSocket_2.54mm:PinSocket_1x15_P2.54mm_Vertical, F.Cu at (279.4, 188.0)
- added ESP2R_1: Conn_01x15_Socket, Connector_PinSocket_2.54mm:PinSocket_1x15_P2.54mm_Vertical, F.Cu at (304.8, 188.0)
- added ESP3L_1: Conn_01x15_Socket, Connector_PinSocket_2.54mm:PinSocket_1x15_P2.54mm_Vertical, F.Cu at (279.4, 99.1)
- added ESP3L_2: Conn_01x15_Socket, Connector_PinSocket_2.54mm:PinSocket_1x15_P2.54mm_Vertical, F.Cu at (269.2, 99.1)
- added ESP3R_1: Conn_01x15_Socket, Connector_PinSocket_2.54mm:PinSocket_1x15_P2.54mm_Vertical, F.Cu at (304.8, 99.1)
- added ESP3R_2: Conn_01x15_Socket, Connector_PinSocket_2.54mm:PinSocket_1x15_P2.54mm_Vertical, F.Cu at (315.0, 99.1)
- added J10: Conn_01x02_Socket, Connector_JST:JST_PH_B2B-PH-K_1x02_P2.00mm_Vertical, F.Cu at (315.0, 190.5)
- added J11: Conn_01x02_Socket, Connector_JST:JST_PH_B2B-PH-K_1x02_P2.00mm_Vertical, F.Cu at (322.6, 200.7)
- added J12: Conn_01x02_Socket, Connector_JST:JST_PH_B2B-PH-K_1x02_P2.00mm_Vertical, F.Cu at (330.2, 203.2)
- added J13: Motor Connect, Connector_Phoenix_MSTB:PhoenixContact_MSTBA_2,5_4-G-5,08_1x04_P5.08mm_Horizontal, F.Cu at (122.8, 349.7)
- added J14: Motor Connect, Connector_Phoenix_MSTB:PhoenixContact_MSTBA_2,5_4-G-5,08_1x04_P5.08mm_Horizontal, F.Cu at (467.4, 264.2)
- added J15: Motor Connect, Connector_Phoenix_MSTB:PhoenixContact_MSTBA_2,5_4-G-5,08_1x04_P5.08mm_Horizontal, F.Cu at (467.4, 213.4)
- added J16: Motor Connect, Connector_Phoenix_MSTB:PhoenixContact_MSTBA_2,5_4-G-5,08_1x04_P5.08mm_Horizontal, F.Cu at (467.4, 162.6)
- added J17: Motor Connect, Connector_Phoenix_MSTB:PhoenixContact_MSTBA_2,5_4-G-5,08_1x04_P5.08mm_Horizontal, F.Cu at (467.4, 111.8)
- added J18: Motor Connect, Connector_Phoenix_MSTB:PhoenixContact_MSTBA_2,5_4-G-5,08_1x04_P5.08mm_Horizontal, F.Cu at (122.8, 197.3)
- added J19: Motor Connect, Connector_Phoenix_MSTB:PhoenixContact_MSTBA_2,5_4-G-5,08_1x04_P5.08mm_Horizontal, F.Cu at (122.8, 248.1)
- added J20: Motor Connect, Connector_Phoenix_MSTB:PhoenixContact_MSTBA_2,5_4-G-5,08_1x04_P5.08mm_Horizontal, F.Cu at (467.4, 315.0)
- added J21: Motor Connect, Connector_Phoenix_MSTB:PhoenixContact_MSTBA_2,5_4-G-5,08_1x04_P5.08mm_Horizontal, F.Cu at (467.4, 365.8)
- added J4: Motor Connect, Connector_Phoenix_MSTB:PhoenixContact_MSTBA_2,5_4-G-5,08_1x04_P5.08mm_Horizontal, F.Cu at (122.8, 95.7)
- added J5: Conn_01x02_Socket, Connector_JST:JST_PH_B2B-PH-K_1x02_P2.00mm_Vertical, F.Cu at (254.0, 162.6)
- added J6: Conn_01x02_Socket, Connector_JST:JST_PH_B2B-PH-K_1x02_P2.00mm_Vertical, F.Cu at (261.6, 160.0)
- added J7: Conn_01x02_Socket, Connector_JST:JST_PH_B2B-PH-K_1x02_P2.00mm_Vertical, F.Cu at (269.2, 157.5)
- added J8: Conn_01x02_Socket, Connector_JST:JST_PH_B2B-PH-K_1x02_P2.00mm_Vertical, F.Cu at (315.0, 198.1)
- added J9: Conn_01x02_Socket, Connector_JST:JST_PH_B2B-PH-K_1x02_P2.00mm_Vertical, F.Cu at (315.0, 147.3)
- added R10: 10k, Resistor_SMD:R_0603_1608Metric, F.Cu at (428.8, 250.6)
- added R11: 69.8k, Resistor_SMD:R_0603_1608Metric, F.Cu at (426.7, 251.9)
- added R12: 15k, Resistor_SMD:R_0603_1608Metric, F.Cu at (424.2, 251.9)
- added R13: 10k, Resistor_SMD:R_0603_1608Metric, F.Cu at (161.5, 362.3)
- added R14: 47.5k, Resistor_SMD:R_0603_1608Metric, F.Cu at (163.6, 361.0)
- added R15: 59k, Resistor_SMD:R_0603_1608Metric, F.Cu at (166.1, 361.0)
- added R16: 10k, Resistor_SMD:R_0603_1608Metric, F.Cu at (161.5, 311.5)
- added R17: 47.5k, Resistor_SMD:R_0603_1608Metric, F.Cu at (163.6, 310.2)
- added R18: 59k, Resistor_SMD:R_0603_1608Metric, F.Cu at (166.1, 310.2)
- added R19: 10k, Resistor_SMD:R_0603_1608Metric, F.Cu at (161.5, 108.3)
- added R20: 21k, Resistor_SMD:R_0603_1608Metric, F.Cu at (163.6, 107.0)
- added R21: 13.7k, Resistor_SMD:R_0603_1608Metric, F.Cu at (166.1, 107.0)
- added R22: 10k, Resistor_SMD:R_0603_1608Metric, F.Cu at (161.5, 159.1)
- added R23: 21k, Resistor_SMD:R_0603_1608Metric, F.Cu at (163.6, 157.8)
- added R24: 13.7k, Resistor_SMD:R_0603_1608Metric, F.Cu at (166.1, 157.8)
- added R25: 10k, Resistor_SMD:R_0603_1608Metric, F.Cu at (161.5, 209.9)
- added R26: 21k, Resistor_SMD:R_0603_1608Metric, F.Cu at (163.6, 208.6)
- added R27: 13.7k, Resistor_SMD:R_0603_1608Metric, F.Cu at (166.1, 208.6)
- added R28: 10k, Resistor_SMD:R_0603_1608Metric, F.Cu at (161.5, 260.7)
- added R29: 21k, Resistor_SMD:R_0603_1608Metric, F.Cu at (163.6, 259.4)
- added R30: 13.7k, Resistor_SMD:R_0603_1608Metric, F.Cu at (166.1, 259.4)
- added R31: 10k, Resistor_SMD:R_0603_1608Metric, F.Cu at (428.8, 301.4)
- added R32: 47.5k, Resistor_SMD:R_0603_1608Metric, F.Cu at (426.7, 302.7)
- added R33: 59k, Resistor_SMD:R_0603_1608Metric, F.Cu at (424.2, 302.7)
- added R34: 10k, Resistor_SMD:R_0603_1608Metric, F.Cu at (428.8, 352.2)
- added R35: 47.5k, Resistor_SMD:R_0603_1608Metric, F.Cu at (426.7, 353.5)
- added R36: 59k, Resistor_SMD:R_0603_1608Metric, F.Cu at (424.2, 353.5)
- added R38: 220E, Resistor_SMD:R_0603_1608Metric, F.Cu at (349.2, 186.2)
- added R39: 4k7, Resistor_SMD:R_0603_1608Metric, F.Cu at (364.5, 182.1)
- added R40: 220E, Resistor_SMD:R_0603_1608Metric, F.Cu at (374.6, 150.7)
- added R41: 4k7, Resistor_SMD:R_0603_1608Metric, F.Cu at (393.7, 149.0)
- added R42: 220E, Resistor_SMD:R_0603_1608Metric, F.Cu at (374.6, 99.9)
- added R43: 4k7, Resistor_SMD:R_0603_1608Metric, F.Cu at (392.4, 98.2)
- added R44: 220E, Resistor_SMD:R_0603_1608Metric, F.Cu at (349.2, 178.6)
- added R45: 4k7, Resistor_SMD:R_0603_1608Metric, F.Cu at (364.5, 176.1)
- added R46: 220E, Resistor_SMD:R_0603_1608Metric, F.Cu at (374.6, 201.5)
- added R47: 4k7, Resistor_SMD:R_0603_1608Metric, F.Cu at (393.7, 199.8)
- added R48: 220E, Resistor_SMD:R_0603_1608Metric, F.Cu at (374.6, 252.3)
- added R49: 4k7, Resistor_SMD:R_0603_1608Metric, F.Cu at (393.7, 250.6)
- added R50: 220E, Resistor_SMD:R_0603_1608Metric, F.Cu at (214.6, 344.6)
- added R51: 4k7, Resistor_SMD:R_0603_1608Metric, F.Cu at (199.4, 348.8)
- added R52: 220E, Resistor_SMD:R_0603_1608Metric, F.Cu at (214.6, 128.7)
- added R53: 4k7, Resistor_SMD:R_0603_1608Metric, F.Cu at (195.6, 130.4)
- added R54: 220E, Resistor_SMD:R_0603_1608Metric, F.Cu at (214.6, 116.0)
- added R55: 4k7, Resistor_SMD:R_0603_1608Metric, F.Cu at (199.4, 120.2)
- added R56: 220E, Resistor_SMD:R_0603_1608Metric, F.Cu at (214.6, 230.3)
- added R57: 4k7, Resistor_SMD:R_0603_1608Metric, F.Cu at (195.6, 232.0)
- added R58: 220E, Resistor_SMD:R_0603_1608Metric, F.Cu at (214.6, 217.6)
- added R59: 4k7, Resistor_SMD:R_0603_1608Metric, F.Cu at (199.4, 221.8)
- added R60: 220E, Resistor_SMD:R_0603_1608Metric, F.Cu at (240.0, 166.8)
- added R61: 4k7, Resistor_SMD:R_0603_1608Metric, F.Cu at (224.8, 171.0)
- added R62: 220E, Resistor_SMD:R_0603_1608Metric, F.Cu at (214.6, 354.8)
- added R63: 4k7, Resistor_SMD:R_0603_1608Metric, F.Cu at (195.6, 356.4)
- added R64: 220E, Resistor_SMD:R_0603_1608Metric, F.Cu at (374.6, 303.1)
- added R65: 4k7, Resistor_SMD:R_0603_1608Metric, F.Cu at (393.7, 301.4)
- added R66: 220E, Resistor_SMD:R_0603_1608Metric, F.Cu at (374.6, 313.2)
- added R67: 4k7, Resistor_SMD:R_0603_1608Metric, F.Cu at (389.9, 309.1)
- added R68: 220E, Resistor_SMD:R_0603_1608Metric, F.Cu at (374.6, 353.9)
- added R69: 4k7, Resistor_SMD:R_0603_1608Metric, F.Cu at (393.7, 352.2)
- added R70: 220E, Resistor_SMD:R_0603_1608Metric, F.Cu at (374.6, 364.0)
- added R71: 4k7, Resistor_SMD:R_0603_1608Metric, F.Cu at (389.9, 359.9)
- added R72: 220E, Resistor_SMD:R_0603_1608Metric, F.Cu at (214.6, 305.6)
- added R73: 4k7, Resistor_SMD:R_0603_1608Metric, F.Cu at (195.6, 305.6)
- added R74: 220E, Resistor_SMD:R_0603_1608Metric, F.Cu at (214.6, 293.8)
- added R75: 4k7, Resistor_SMD:R_0603_1608Metric, F.Cu at (199.4, 298.0)
- added R76: 220E, Resistor_SMD:R_0603_1608Metric, F.Cu at (290.0, 316.2)
- added R77: 4k7, Resistor_SMD:R_0603_1608Metric, F.Cu at (294.2, 331.5)
- added U10: PC817, Package_DIP:DIP-4_W7.62mm, F.Cu at (210.8, 297.2)
- added U11: 6N137, 6n137:DIP762W60P254L968H450Q8N, F.Cu at (207.0, 356.9)
- added U12: PC817, Package_DIP:DIP-4_W7.62mm, F.Cu at (293.4, 320.0)
- added U13: PC817, Package_DIP:DIP-4_W7.62mm, F.Cu at (353.1, 182.9)
- added U14: 6N137, 6n137:DIP762W60P254L968H450Q8N, F.Cu at (382.3, 148.6)
- added U15: 6N137, 6n137:DIP762W60P254L968H450Q8N, F.Cu at (382.3, 97.8)
- added U16: PC817, Package_DIP:DIP-4_W7.62mm, F.Cu at (353.1, 175.3)
- added U17: 6N137, 6n137:DIP762W60P254L968H450Q8N, F.Cu at (382.3, 199.4)
- added U18: 6N137, 6n137:DIP762W60P254L968H450Q8N, F.Cu at (382.3, 250.2)
- added U19: PC817, Package_DIP:DIP-4_W7.62mm, F.Cu at (210.8, 348.0)
- added U20: 6N137, 6n137:DIP762W60P254L968H450Q8N, F.Cu at (382.3, 301.0)
- added U21: PC817, Package_DIP:DIP-4_W7.62mm, F.Cu at (378.5, 309.9)
- added U3: PC817, Package_DIP:DIP-4_W7.62mm, F.Cu at (210.8, 221.0)
- added U5: PC817, Package_DIP:DIP-4_W7.62mm, F.Cu at (236.2, 170.2)
- added U7: 6N137, 6n137:DIP762W60P254L968H450Q8N, F.Cu at (382.3, 351.8)
- added U8: PC817, Package_DIP:DIP-4_W7.62mm, F.Cu at (378.5, 360.7)
- added U9: 6N137, 6n137:DIP762W60P254L968H450Q8N, F.Cu at (207.0, 306.1)
- added UDRIVE1: DRV8434PWPR, footprints:TSSOP_34PWPR_TEX, F.Cu at (155.4, 255.7)
- added UDRIVE2: DRV8434PWPR, footprints:TSSOP_34PWPR_TEX, F.Cu at (155.4, 204.9)
- added UDRIVE3: DRV8434PWPR, footprints:TSSOP_34PWPR_TEX, F.Cu at (155.4, 154.1)
- added UDRIVE4: DRV8434PWPR, footprints:TSSOP_34PWPR_TEX, F.Cu at (155.4, 103.3)
- added ULIFT1: DRV8434PWPR, footprints:TSSOP_34PWPR_TEX, F.Cu at (434.8, 103.3)
- added ULIFT2: DRV8434PWPR, footprints:TSSOP_34PWPR_TEX, F.Cu at (434.8, 154.1)
- added ULIFT3: DRV8434PWPR, footprints:TSSOP_34PWPR_TEX, F.Cu at (434.8, 204.9)
- added ULIFT4: DRV8434PWPR, footprints:TSSOP_34PWPR_TEX, F.Cu at (434.8, 255.7)
- added UTURN1: DRV8434PWPR, footprints:TSSOP_34PWPR_TEX, F.Cu at (155.4, 306.5)
- added UTURN2: DRV8434PWPR, footprints:TSSOP_34PWPR_TEX, F.Cu at (434.8, 306.5)
- added UTURN3: DRV8434PWPR, footprints:TSSOP_34PWPR_TEX, F.Cu at (155.4, 357.3)
- added UTURN4: DRV8434PWPR, footprints:TSSOP_34PWPR_TEX, F.Cu at (434.8, 357.3)
- C1, C4: footprint Capacitor_SMD:C_0603_1608Metric_Pad1.08x0.95mm_HandSolder -> Capacitor_SMD:C_0603_1608Metric
- C2: value 220n -> 1u; footprint Capacitor_SMD:C_0603_1608Metric_Pad1.08x0.95mm_HandSolder -> Capacitor_SMD:C_0603_1608Metric
- C3: value 0.01u -> 220n; footprint Capacitor_SMD:C_0603_1608Metric_Pad1.08x0.95mm_HandSolder -> Capacitor_SMD:C_0603_1608Metric
- C5: value 100u -> 0.01u; footprint Capacitor_THT:CP_Radial_D8.0mm_P3.50mm -> Capacitor_SMD:C_0603_1608Metric
- C6: value 1u -> 22n; footprint Capacitor_SMD:C_0603_1608Metric_Pad1.08x0.95mm_HandSolder -> Capacitor_SMD:C_0603_1608Metric
- C7: value 0.1u -> 1u; footprint Capacitor_SMD:C_0603_1608Metric_Pad1.08x0.95mm_HandSolder -> Capacitor_SMD:C_0603_1608Metric
- J2: value PWR & DATA Connect -> Motor Connect; footprint Connector_Phoenix_MSTB:PhoenixContact_MSTBA_2,5_5-G-5,08_1x05_P5.08mm_Horizontal -> Connector_Phoenix_MSTB:PhoenixContact_MSTBA_2,5_4-G-5,08_1x04_P5.08mm_Horizontal
- R1: footprint Resistor_SMD:R_0603_1608Metric_Pad0.98x0.95mm_HandSolder -> Resistor_SMD:R_0603_1608Metric
- R2: value 10k -> 69.8k; footprint Resistor_SMD:R_0603_1608Metric_Pad0.98x0.95mm_HandSolder -> Resistor_SMD:R_0603_1608Metric
- R3: value 10k -> 15k; footprint Resistor_SMD:R_0603_1608Metric_Pad0.98x0.95mm_HandSolder -> Resistor_SMD:R_0603_1608Metric
- R4: value 220E -> 10k; footprint Resistor_SMD:R_0603_1608Metric_Pad0.98x0.95mm_HandSolder -> Resistor_SMD:R_0603_1608Metric
- R5: value 4k7 -> 69.8k; footprint Resistor_SMD:R_0603_1608Metric_Pad0.98x0.95mm_HandSolder -> Resistor_SMD:R_0603_1608Metric
- R6: value 220E -> 15k; footprint Resistor_SMD:R_0603_1608Metric_Pad0.98x0.95mm_HandSolder -> Resistor_SMD:R_0603_1608Metric
- R7: value 4k7 -> 10k; footprint Resistor_SMD:R_0603_1608Metric_Pad0.98x0.95mm_HandSolder -> Resistor_SMD:R_0603_1608Metric
- R8: value 220E -> 69.8k; footprint Resistor_SMD:R_0603_1608Metric_Pad0.98x0.95mm_HandSolder -> Resistor_SMD:R_0603_1608Metric
- R9: value 4k7 -> 15k; footprint Resistor_SMD:R_0603_1608Metric_Pad0.98x0.95mm_HandSolder -> Resistor_SMD:R_0603_1608Metric
- U2: value PC817 -> 6N137; footprint Package_DIP:DIP-4_W7.62mm -> 6n137:DIP762W60P254L968H450Q8N
- U4: footprint Package_DIP:DIP-8_W7.62mm -> 6n137:DIP762W60P254L968H450Q8N
- moved J3 316.6 mm to (289.6, 367.8)
- moved C5 297.3 mm to (440.2, 99.3), turned to -90 degrees
- moved C4 296.7 mm to (440.2, 107.2)
- moved C3 296.1 mm to (438.4, 109.5), turned to 0 degrees
- moved R9 294.5 mm to (424.2, 201.1)
- moved R7 293.2 mm to (428.8, 199.8), turned to -90 degrees
- moved C2 287.9 mm to (432.6, 96.5), turned to 0 degrees
- moved C6 287.8 mm to (429.3, 158.8), turned to 90 degrees
- moved R8 277.8 mm to (426.7, 201.1), turned to 90 degrees
- moved C7 276.6 mm to (432.6, 147.3), turned to 0 degrees
- moved C1 276.0 mm to (429.3, 108.0), turned to 90 degrees
- moved R1 274.4 mm to (428.8, 98.2), turned to -90 degrees
- moved R5 273.9 mm to (426.7, 150.3), turned to 90 degrees
- moved R4 271.1 mm to (428.8, 149.0), turned to -90 degrees
- moved R6 269.9 mm to (424.2, 150.3), turned to -90 degrees
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Connections:
- net /VREF renamed Net-(ULIFT1-VREF)
- C1 pad 1: /CPH -> Net-(ULIFT1-CPH)
- C1 pad 2: /CPL -> Net-(ULIFT1-CPL)
- C2 pad 1: /VCP -> +DVDD_L1
- C2 pad 2: +BATT -> GND
- C3 pad 1: +BATT -> Net-(ULIFT1-VCP)
- C3 pad 2: GND -> +BATT
- C6 pad 1: +5V -> Net-(ULIFT2-CPH)
- C6 pad 2: GND -> Net-(ULIFT2-CPL)
- C7 pad 1: +5V -> +DVDD_L2
- J1 pad 1: /AOUT1 -> /AOUT1_T1
- J1 pad 2: /AOUT2 -> /AOUT2_T1
- J1 pad 3: /BOUT2 -> /BOUT2_T1
- J1 pad 4: /BOUT1 -> /BOUT1_T1
- J2 pad 1: +5V -> /AOUT1_D3
- J2 pad 2: GND -> /AOUT2_D3
- J2 pad 3: /PUL_ESP -> /BOUT2_D3
- J2 pad 4: /DIR_ESP -> /BOUT1_D3
- R1 pad 1: +5V -> +DVDD_L1
- R1 pad 2: /FAULT -> Net-(ULIFT1-nFAULT)
- R2 pad 2: +5V -> +DVDD_L1
- R4 pad 1: GND -> +DVDD_L2
- R4 pad 2: Net-(R4-Pad2) -> Net-(ULIFT2-nFAULT)
- R5 pad 1: /DIR -> Net-(ULIFT2-VREF)
- R5 pad 2: +5V -> +DVDD_L2
- R6 pad 2: Net-(R6-Pad2) -> Net-(ULIFT2-VREF)
- R7 pad 1: /PUL -> +DVDD_L3
- R7 pad 2: +5V -> Net-(ULIFT3-nFAULT)
- R8 pad 1: GND -> Net-(ULIFT3-VREF)
- R8 pad 2: Net-(U4-C) -> +DVDD_L3
- R9 pad 1: /ENA -> GND
- R9 pad 2: +5V -> Net-(ULIFT3-VREF)
- U2 pad 1: /DIR_ESP -> unconnected-(U2-NC-Pad1)
- U2 pad 2: Net-(R4-Pad2) -> /ESPs/FRONT_DRIVE_PUL_ESP
- U2 pad 3: GND -> Net-(U2-C)
- U2 pad 4: /DIR -> unconnected-(U2-NC-Pad4)
- U4 pad 2: /PUL_ESP -> /ESPs/BACK_DRIVE_PUL_ESP
- U4 pad 6: /PUL -> /BACK_DRIVE_PUL
- U6 pad 1: /ENA_ESP -> /ESPs/BACK_DRIVE_DIR_ESP
- U6 pad 2: Net-(R6-Pad2) -> Net-(R54-Pad2)
- U6 pad 4: /ENA -> /BACK_DRIVE_DIR
Routing:
- net /M1: track 33.4 -> 0.00 mm
- net +5V: track 5.84 -> 38.1 mm, vias 11 -> 0
- net /ESPs/Limit_2_18: track 0.00 -> 25.4 mm
- net /ESPs/Limit_1_25: track 0.00 -> 25.4 mm
- net /ENA: track 24.6 -> 0.00 mm
- net /M0: track 24.1 -> 0.00 mm
- net GNDD: track 0.00 -> 20.3 mm
- net /DIR: track 17.9 -> 0.00 mm
- net /ESPs/Limit_2_19: track 0.00 -> 17.8 mm
- net /ESPs/Limit_1_33: track 0.00 -> 17.8 mm
- net /PUL: track 16.6 -> 0.00 mm
- net /ENA_ESP: track 15.3 -> 0.00 mm
- net GND: track 18.2 -> 5.28 mm, vias 126 -> 0
- net /DIR_ESP: track 12.3 -> 0.00 mm
- net /PUL_ESP: track 10.4 -> 0.00 mm
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- added copper zone on In1.Cu, net GNDD
- removed copper zone on F.Cu, net +5V
- removed copper zone on F.Cu, net +BATT
- removed copper zone on In2.Cu, net +BATT
- removed copper zone on F.Cu, net /AOUT1
- removed copper zone on F.Cu, net /AOUT2
- removed copper zone on F.Cu, net /BOUT1
- removed copper zone on F.Cu, net /BOUT2
- removed copper zone on F.Cu, net GND
Other:
- board size 75 x 46.8 mm -> 381 x 304.8 mm
- board text removed: "1 Z 0"
- board text removed: "M0:"
- board text removed: "M0=0, M1=1 -> 1/4 M0=1, M1=1 -> 1/8 M0=Z, M1=1 -> 1/6"
- board text removed: "M1:"
- board text removed: "NEON CARROT STEPPER MOTOR DRIVER"
