File: KiCad/12_Driver_Board/12_Driver_Board.kicad_sch (KiCad schematic)
At the start: 135 parts, among them J1 Motor Connect, J13 Motor Connect, J14 Motor Connect, J15 Motor Connect, J16 Motor Connect, J17 Motor Connect, J18 Motor Connect, J19 Motor Connect, J2 Motor Connect, J20 Motor Connect, J21 Motor Connect, J3 Battery Connect, J4 Motor Connect, SW1 SW_SPDT_MSM, SW2 SW_SPDT_MSM, U1 DRV8434PWPR, U22 DRV8434PWPR, U23 DRV8434PWPR, U24 DRV8434PWPR, U25 DRV8434PWPR, U26 DRV8434PWPR, U27 DRV8434PWPR, U28 DRV8434PWPR, U29 DRV8434PWPR, U30 DRV8434PWPR, U31 DRV8434PWPR, U32 DRV8434PWPR

Commit message: Adding Cad files
Parts:
- removed C17, C23, C29, C35, C36, C47, C5, C53, C59, C60, C71, C72: 100u, Capacitor_THT:CP_Radial_D8.0mm_P3.50mm, symbol Device:C_Polarized
- added JBUCK5_LOGIC1, JBUCK5_MOTOR1: Conn_01x04_Pin, symbol Connector:Conn_01x04_Pin
- UDRIVE1: renamed from U30; footprint DRV8434PWPR:TSSOP_34PWPR_TEX -> footprints:TSSOP_34PWPR_TEX
- UDRIVE2: renamed from U29; footprint DRV8434PWPR:TSSOP_34PWPR_TEX -> footprints:TSSOP_34PWPR_TEX
- UDRIVE3: renamed from U22; footprint DRV8434PWPR:TSSOP_34PWPR_TEX -> footprints:TSSOP_34PWPR_TEX
- UDRIVE4: renamed from U23; footprint DRV8434PWPR:TSSOP_34PWPR_TEX -> footprints:TSSOP_34PWPR_TEX
- ULIFT1: renamed from U1; footprint DRV8434PWPR:TSSOP_34PWPR_TEX -> footprints:TSSOP_34PWPR_TEX
- ULIFT2: renamed from U24; footprint DRV8434PWPR:TSSOP_34PWPR_TEX -> footprints:TSSOP_34PWPR_TEX
- ULIFT3: renamed from U25; footprint DRV8434PWPR:TSSOP_34PWPR_TEX -> footprints:TSSOP_34PWPR_TEX
- ULIFT4: renamed from U26; footprint DRV8434PWPR:TSSOP_34PWPR_TEX -> footprints:TSSOP_34PWPR_TEX
- UTURN1: renamed from U28; footprint DRV8434PWPR:TSSOP_34PWPR_TEX -> footprints:TSSOP_34PWPR_TEX
- UTURN2: renamed from U31; footprint DRV8434PWPR:TSSOP_34PWPR_TEX -> footprints:TSSOP_34PWPR_TEX
- UTURN3: renamed from U27; footprint DRV8434PWPR:TSSOP_34PWPR_TEX -> footprints:TSSOP_34PWPR_TEX
- UTURN4: renamed from U32; footprint DRV8434PWPR:TSSOP_34PWPR_TEX -> footprints:TSSOP_34PWPR_TEX
- renumbered C31 to C10, C45 to C11, C43 to C12, C41 to C13, C37 to C14, C39 to C15, C46 to C16, C44 to C17, C42 to C18, C38 to C19, C6 to C2, C40 to C20, C52 to C21, C51 to C22, C50 to C23, C48 to C24, C49 to C25, C58 to C26, C57 to C27, C56 to C28, C54 to C29, C2 to C3, C55 to C30, C28 to C31, C27 to C32, C26 to C33, C24 to C34, C25 to C35, C22 to C36, C21 to C37, C20 to C38, C18 to C39, C3 to C4, C19 to C40, C69 to C41, C67 to C42, C65 to C43, C61 to C44, C63 to C45, C70 to C46, C68 to C47, C66 to C48, C62 to C49, C4 to C5, C64 to C50, C81 to C51, C79 to C52, C77 to C53, C73 to C54, C75 to C55, C82 to C56, C80 to C57, C78 to C58, C74 to C59, C34 to C6, C76 to C60, C33 to C7, C32 to C8, C30 to C9, R54 to R10, R57 to R11, R58 to R12, R59 to R13, R60 to R14, R61 to R15, R62 to R16, R63 to R17, R64 to R18, R47 to R19, R48 to R20, R49 to R21, R44 to R22, R45 to R23, R46 to R24, R65 to R25, R67 to R26, R68 to R27, R66 to R28, R69 to R29, R70 to R30, R71 to R31, R73 to R32, R74 to R33, R72 to R34, R75 to R35, R76 to R36, R50 to R4, R51 to R5, R52 to R6, R53 to R7, R55 to R8, R56 to R9
Connections:
- net LIFT1_DIR is gone; now on net LIFT_DIR: ULIFT1.24 (DIR)
- net LIFT2_DIR is gone; now on net LIFT_DIR: ULIFT2.24 (DIR)
- net LIFT3_DIR is gone; now on net LIFT_DIR: ULIFT3.24 (DIR)
- net LIFT4_DIR is gone; now on net LIFT_DIR: ULIFT4.24 (DIR)
- net +5V: now also JBUCK5_MOTOR1.4 (Pin_4); no longer C12.1, C17.1, C2.1, C22.1, C27.1, C32.1, C37.1, C42.1, C47.1, C52.1, C57.1, C7.1, R1.1, R10.1, R11.2, R13.1, R14.2, R16.1, R17.2, R19.1, R2.2, R20.2, R22.1, R23.2, R25.1, R26.2, R28.1, R29.2, R31.1, R32.2, R34.1, R35.2, R4.1, R5.2, R7.1, R8.2, UDRIVE1.15 (DVDD), UDRIVE1.19 (TOFF), UDRIVE1.20 (DECAY1), UDRIVE1.26 (nSLEEP), UDRIVE2.15 (DVDD), UDRIVE2.19 (TOFF), UDRIVE2.20 (DECAY1), UDRIVE2.26 (nSLEEP), UDRIVE3.15 (DVDD), UDRIVE3.19 (TOFF), UDRIVE3.20 (DECAY1), UDRIVE3.26 (nSLEEP), UDRIVE4.15 (DVDD), UDRIVE4.19 (TOFF), UDRIVE4.20 (DECAY1), UDRIVE4.26 (nSLEEP), ULIFT1.15 (DVDD), ULIFT1.19 (TOFF), ULIFT1.20 (DECAY1), ULIFT1.26 (nSLEEP), ULIFT2.15 (DVDD), ULIFT2.19 (TOFF), ULIFT2.20 (DECAY1), ULIFT2.26 (nSLEEP), ULIFT3.15 (DVDD), ULIFT3.19 (TOFF), ULIFT3.20 (DECAY1), ULIFT3.26 (nSLEEP), ULIFT4.15 (DVDD), ULIFT4.19 (TOFF), ULIFT4.20 (DECAY1), ULIFT4.26 (nSLEEP), UTURN1.15 (DVDD), UTURN1.19 (TOFF), UTURN1.20 (DECAY1), UTURN1.26 (nSLEEP), UTURN2.15 (DVDD), UTURN2.19 (TOFF), UTURN2.20 (DECAY1), UTURN2.26 (nSLEEP), UTURN3.15 (DVDD), UTURN3.19 (TOFF), UTURN3.20 (DECAY1), UTURN3.26 (nSLEEP), UTURN4.15 (DVDD), UTURN4.19 (TOFF), UTURN4.20 (DECAY1), UTURN4.26 (nSLEEP)
- net GND: now also JBUCK5_MOTOR1.1 (Pin_1)
- net LIFT1_PUL: now also ULIFT1.23 (STEP)
- net LIFT4_PUL: no longer ULIFT1.23 (STEP)
- removed net AOUT1: J1.1 (Pin_1), J13.1 (Pin_1), J14.1 (Pin_1), J15.1 (Pin_1), J16.1 (Pin_1), J17.1 (Pin_1), J18.1 (Pin_1), J19.1 (Pin_1), J2.1 (Pin_1), J20.1 (Pin_1), J21.1 (Pin_1), J4.1 (Pin_1), UDRIVE1.4 (AOUT1), UDRIVE1.5 (AOUT1), UDRIVE2.4 (AOUT1), UDRIVE2.5 (AOUT1), UDRIVE3.4 (AOUT1), UDRIVE3.5 (AOUT1), UDRIVE4.4 (AOUT1), UDRIVE4.5 (AOUT1), ULIFT1.4 (AOUT1), ULIFT1.5 (AOUT1), ULIFT2.4 (AOUT1), ULIFT2.5 (AOUT1), ULIFT3.4 (AOUT1), ULIFT3.5 (AOUT1), ULIFT4.4 (AOUT1), ULIFT4.5 (AOUT1), UTURN1.4 (AOUT1), UTURN1.5 (AOUT1), UTURN2.4 (AOUT1), UTURN2.5 (AOUT1), UTURN3.4 (AOUT1), UTURN3.5 (AOUT1), UTURN4.4 (AOUT1), UTURN4.5 (AOUT1)
- removed net AOUT2: J1.2 (Pin_2), J13.2 (Pin_2), J14.2 (Pin_2), J15.2 (Pin_2), J16.2 (Pin_2), J17.2 (Pin_2), J18.2 (Pin_2), J19.2 (Pin_2), J2.2 (Pin_2), J20.2 (Pin_2), J21.2 (Pin_2), J4.2 (Pin_2), UDRIVE1.6 (AOUT2), UDRIVE1.7 (AOUT2), UDRIVE2.6 (AOUT2), UDRIVE2.7 (AOUT2), UDRIVE3.6 (AOUT2), UDRIVE3.7 (AOUT2), UDRIVE4.6 (AOUT2), UDRIVE4.7 (AOUT2), ULIFT1.6 (AOUT2), ULIFT1.7 (AOUT2), ULIFT2.6 (AOUT2), ULIFT2.7 (AOUT2), ULIFT3.6 (AOUT2), ULIFT3.7 (AOUT2), ULIFT4.6 (AOUT2), ULIFT4.7 (AOUT2), UTURN1.6 (AOUT2), UTURN1.7 (AOUT2), UTURN2.6 (AOUT2), UTURN2.7 (AOUT2), UTURN3.6 (AOUT2), UTURN3.7 (AOUT2), UTURN4.6 (AOUT2), UTURN4.7 (AOUT2)
- removed net BOUT1: J1.4 (Pin_4), J13.4 (Pin_4), J14.4 (Pin_4), J15.4 (Pin_4), J16.4 (Pin_4), J17.4 (Pin_4), J18.4 (Pin_4), J19.4 (Pin_4), J2.4 (Pin_4), J20.4 (Pin_4), J21.4 (Pin_4), J4.4 (Pin_4), UDRIVE1.10 (BOUT1), UDRIVE1.11 (BOUT1), UDRIVE2.10 (BOUT1), UDRIVE2.11 (BOUT1), UDRIVE3.10 (BOUT1), UDRIVE3.11 (BOUT1), UDRIVE4.10 (BOUT1), UDRIVE4.11 (BOUT1), ULIFT1.10 (BOUT1), ULIFT1.11 (BOUT1), ULIFT2.10 (BOUT1), ULIFT2.11 (BOUT1), ULIFT3.10 (BOUT1), ULIFT3.11 (BOUT1), ULIFT4.10 (BOUT1), ULIFT4.11 (BOUT1), UTURN1.10 (BOUT1), UTURN1.11 (BOUT1), UTURN2.10 (BOUT1), UTURN2.11 (BOUT1), UTURN3.10 (BOUT1), UTURN3.11 (BOUT1), UTURN4.10 (BOUT1), UTURN4.11 (BOUT1)
- removed net BOUT2: J1.3 (Pin_3), J13.3 (Pin_3), J14.3 (Pin_3), J15.3 (Pin_3), J16.3 (Pin_3), J17.3 (Pin_3), J18.3 (Pin_3), J19.3 (Pin_3), J2.3 (Pin_3), J20.3 (Pin_3), J21.3 (Pin_3), J4.3 (Pin_3), UDRIVE1.8 (BOUT2), UDRIVE1.9 (BOUT2), UDRIVE2.8 (BOUT2), UDRIVE2.9 (BOUT2), UDRIVE3.8 (BOUT2), UDRIVE3.9 (BOUT2), UDRIVE4.8 (BOUT2), UDRIVE4.9 (BOUT2), ULIFT1.8 (BOUT2), ULIFT1.9 (BOUT2), ULIFT2.8 (BOUT2), ULIFT2.9 (BOUT2), ULIFT3.8 (BOUT2), ULIFT3.9 (BOUT2), ULIFT4.8 (BOUT2), ULIFT4.9 (BOUT2), UTURN1.8 (BOUT2), UTURN1.9 (BOUT2), UTURN2.8 (BOUT2), UTURN2.9 (BOUT2), UTURN3.8 (BOUT2), UTURN3.9 (BOUT2), UTURN4.8 (BOUT2), UTURN4.9 (BOUT2)
- removed net CPH: C1.1, C11.1, C16.1, C21.1, C26.1, C31.1, C36.1, C41.1, C46.1, C51.1, C56.1, C6.1, UDRIVE1.28 (CPH), UDRIVE2.28 (CPH), UDRIVE3.28 (CPH), UDRIVE4.28 (CPH), ULIFT1.28 (CPH), ULIFT2.28 (CPH), ULIFT3.28 (CPH), ULIFT4.28 (CPH), UTURN1.28 (CPH), UTURN2.28 (CPH), UTURN3.28 (CPH), UTURN4.28 (CPH)
- removed net CPL: C1.2, C11.2, C16.2, C21.2, C26.2, C31.2, C36.2, C41.2, C46.2, C51.2, C56.2, C6.2, UDRIVE1.27 (CPL), UDRIVE2.27 (CPL), UDRIVE3.27 (CPL), UDRIVE4.27 (CPL), ULIFT1.27 (CPL), ULIFT2.27 (CPL), ULIFT3.27 (CPL), ULIFT4.27 (CPL), UTURN1.27 (CPL), UTURN2.27 (CPL), UTURN3.27 (CPL), UTURN4.27 (CPL)
- removed net FAULT: R1.2, R10.2, R13.2, R16.2, R19.2, R22.2, R25.2, R28.2, R31.2, R34.2, R4.2, R7.2, UDRIVE1.16 (nFAULT), UDRIVE2.16 (nFAULT), UDRIVE3.16 (nFAULT), UDRIVE4.16 (nFAULT), ULIFT1.16 (nFAULT), ULIFT2.16 (nFAULT), ULIFT3.16 (nFAULT), ULIFT4.16 (nFAULT), UTURN1.16 (nFAULT), UTURN2.16 (nFAULT), UTURN3.16 (nFAULT), UTURN4.16 (nFAULT)
- removed net VCP: C13.1, C18.1, C23.1, C28.1, C3.1, C33.1, C38.1, C43.1, C48.1, C53.1, C58.1, C8.1, UDRIVE1.1 (VCP), UDRIVE2.1 (VCP), UDRIVE3.1 (VCP), UDRIVE4.1 (VCP), ULIFT1.1 (VCP), ULIFT2.1 (VCP), ULIFT3.1 (VCP), ULIFT4.1 (VCP), UTURN1.1 (VCP), UTURN2.1 (VCP), UTURN3.1 (VCP), UTURN4.1 (VCP)
- removed net VREF: R11.1, R12.2, R14.1, R15.2, R17.1, R18.2, R2.1, R20.1, R21.2, R23.1, R24.2, R26.1, R27.2, R29.1, R3.2, R30.2, R32.1, R33.2, R35.1, R36.2, R5.1, R6.2, R8.1, R9.2, UDRIVE1.17 (VREF), UDRIVE2.17 (VREF), UDRIVE3.17 (VREF), UDRIVE4.17 (VREF), ULIFT1.17 (VREF), ULIFT2.17 (VREF), ULIFT3.17 (VREF), ULIFT4.17 (VREF), UTURN1.17 (VREF), UTURN2.17 (VREF), UTURN3.17 (VREF), UTURN4.17 (VREF)
- new net: C23.1, UTURN3.1 (VCP)
- new net: R13.2, UTURN3.16 (nFAULT)
- new net: R14.1, R15.2, UTURN3.17 (VREF)
- new net: C21.2, UTURN3.27 (CPL)
- new net: C21.1, UTURN3.28 (CPH)
- new net: C8.1, ULIFT2.1 (VCP)
- new net: C36.1, UDRIVE3.28 (CPH)
- new net: C36.2, UDRIVE3.27 (CPL)
- new net: C48.1, UDRIVE1.1 (VCP)
- new net: R28.2, UDRIVE1.16 (nFAULT)
- new net: R29.1, R30.2, UDRIVE1.17 (VREF)
- new net: C46.2, UDRIVE1.27 (CPL)
- new net: C46.1, UDRIVE1.28 (CPH)
- new net: R4.2, ULIFT2.16 (nFAULT)
- new net: R5.1, R6.2, ULIFT2.17 (VREF)
- new net: C6.2, ULIFT2.27 (CPL)
- new net: C6.1, ULIFT2.28 (CPH)
- new net: R20.1, R21.2, UDRIVE4.17 (VREF)
- new net: C11.1, ULIFT3.28 (CPH)
- new net: C11.2, ULIFT3.27 (CPL)
- new net: C18.1, ULIFT4.1 (VCP)
- new net: R10.2, ULIFT4.16 (nFAULT)
- new net: R11.1, R12.2, ULIFT4.17 (VREF)
- new net: C16.2, ULIFT4.27 (CPL)
- new net: C16.1, ULIFT4.28 (CPH)
- new net: R23.1, R24.2, UDRIVE3.17 (VREF)
- new net: C31.1, UDRIVE4.28 (CPH)
- new net: C31.2, UDRIVE4.27 (CPL)
- new net: C28.1, UTURN1.1 (VCP)
- new net: R16.2, UTURN1.16 (nFAULT)
- new net: R17.1, R18.2, UTURN1.17 (VREF)
- new net: C26.2, UTURN1.27 (CPL)
- new net: C26.1, UTURN1.28 (CPH)
- new net: R1.2, ULIFT1.16 (nFAULT)
- new net: C56.1, UTURN4.28 (CPH)
- new net: C56.2, UTURN4.27 (CPL)
- new net: C38.1, UDRIVE3.1 (VCP)
- new net: C51.1, UTURN2.28 (CPH)
- new net: C51.2, UTURN2.27 (CPL)
- new net: R19.2, UDRIVE4.16 (nFAULT)
- new net: R26.1, R27.2, UDRIVE2.17 (VREF)
- new net: R32.1, R33.2, UTURN2.17 (VREF)
- new net: R2.1, R3.2, ULIFT1.17 (VREF)
- new net: C58.1, UTURN4.1 (VCP)
- new net: R8.1, R9.2, ULIFT3.17 (VREF)
- new net: C43.1, UDRIVE2.1 (VCP)
- new net: C3.1, ULIFT1.1 (VCP)
- new net: R35.1, R36.2, UTURN4.17 (VREF)
- new net: R31.2, UTURN2.16 (nFAULT)
- new net: R22.2, UDRIVE3.16 (nFAULT)
- new net: R25.2, UDRIVE2.16 (nFAULT)
- new net: C13.1, ULIFT3.1 (VCP)
- new net: R7.2, ULIFT3.16 (nFAULT)
- new net: C1.1, ULIFT1.28 (CPH)
- new net: C1.2, ULIFT1.27 (CPL)
- new net: R34.2, UTURN4.16 (nFAULT)
- new net: C33.1, UDRIVE4.1 (VCP)
- new net: C41.2, UDRIVE2.27 (CPL)
- new net: C41.1, UDRIVE2.28 (CPH)
- new net: C53.1, UTURN2.1 (VCP)
- new net +5VD: JBUCK5_LOGIC1.4 (Pin_4)
- new net +DVDD_D1: C47.1, R28.1, R29.2, UDRIVE1.15 (DVDD), UDRIVE1.19 (TOFF), UDRIVE1.20 (DECAY1), UDRIVE1.26 (nSLEEP)
- new net +DVDD_D2: C42.1, R25.1, R26.2, UDRIVE2.15 (DVDD), UDRIVE2.19 (TOFF), UDRIVE2.20 (DECAY1), UDRIVE2.26 (nSLEEP)
- new net +DVDD_D3: C37.1, R22.1, R23.2, UDRIVE3.15 (DVDD), UDRIVE3.19 (TOFF), UDRIVE3.20 (DECAY1), UDRIVE3.26 (nSLEEP)
- new net +DVDD_D4: C32.1, R19.1, R20.2, UDRIVE4.15 (DVDD), UDRIVE4.19 (TOFF), UDRIVE4.20 (DECAY1), UDRIVE4.26 (nSLEEP)
- new net +DVDD_L1: C2.1, R1.1, R2.2, ULIFT1.15 (DVDD), ULIFT1.19 (TOFF), ULIFT1.20 (DECAY1), ULIFT1.26 (nSLEEP)
- new net +DVDD_L2: C7.1, R4.1, R5.2, ULIFT2.15 (DVDD), ULIFT2.19 (TOFF), ULIFT2.20 (DECAY1), ULIFT2.26 (nSLEEP)
- new net +DVDD_L3: C12.1, R7.1, R8.2, ULIFT3.15 (DVDD), ULIFT3.19 (TOFF), ULIFT3.20 (DECAY1), ULIFT3.26 (nSLEEP)
- new net +DVDD_L4: C17.1, R10.1, R11.2, ULIFT4.15 (DVDD), ULIFT4.19 (TOFF), ULIFT4.20 (DECAY1), ULIFT4.26 (nSLEEP)
- new net +DVDD_T1: C27.1, R16.1, R17.2, UTURN1.15 (DVDD), UTURN1.19 (TOFF), UTURN1.20 (DECAY1), UTURN1.26 (nSLEEP)
- new net +DVDD_T2: C52.1, R31.1, R32.2, UTURN2.15 (DVDD), UTURN2.19 (TOFF), UTURN2.20 (DECAY1), UTURN2.26 (nSLEEP)
- new net +DVDD_T3: C22.1, R13.1, R14.2, UTURN3.15 (DVDD), UTURN3.19 (TOFF), UTURN3.20 (DECAY1), UTURN3.26 (nSLEEP)
- new net +DVDD_T4: C57.1, R34.1, R35.2, UTURN4.15 (DVDD), UTURN4.19 (TOFF), UTURN4.20 (DECAY1), UTURN4.26 (nSLEEP)
- new net AOUT1_D1: J19.1 (Pin_1), UDRIVE1.4 (AOUT1), UDRIVE1.5 (AOUT1)
- new net AOUT1_D2: J18.1 (Pin_1), UDRIVE2.4 (AOUT1), UDRIVE2.5 (AOUT1)
- new net AOUT1_D3: J2.1 (Pin_1), UDRIVE3.4 (AOUT1), UDRIVE3.5 (AOUT1)
- new net AOUT1_D4: J4.1 (Pin_1), UDRIVE4.4 (AOUT1), UDRIVE4.5 (AOUT1)
- new net AOUT1_L1: J17.1 (Pin_1), ULIFT1.4 (AOUT1), ULIFT1.5 (AOUT1)
- new net AOUT1_L2: J16.1 (Pin_1), ULIFT2.4 (AOUT1), ULIFT2.5 (AOUT1)
- new net AOUT1_L3: J15.1 (Pin_1), ULIFT3.4 (AOUT1), ULIFT3.5 (AOUT1)
- new net AOUT1_L4: J14.1 (Pin_1), ULIFT4.4 (AOUT1), ULIFT4.5 (AOUT1)
- new net AOUT1_T1: J1.1 (Pin_1), UTURN1.4 (AOUT1), UTURN1.5 (AOUT1)
- new net AOUT1_T2: J20.1 (Pin_1), UTURN2.4 (AOUT1), UTURN2.5 (AOUT1)
- new net AOUT1_T3: J13.1 (Pin_1), UTURN3.4 (AOUT1), UTURN3.5 (AOUT1)
- new net AOUT1_T4: J21.1 (Pin_1), UTURN4.4 (AOUT1), UTURN4.5 (AOUT1)
- new net AOUT2_D1: J19.2 (Pin_2), UDRIVE1.6 (AOUT2), UDRIVE1.7 (AOUT2)
- new net AOUT2_D2: J18.2 (Pin_2), UDRIVE2.6 (AOUT2), UDRIVE2.7 (AOUT2)
- new net AOUT2_D3: J2.2 (Pin_2), UDRIVE3.6 (AOUT2), UDRIVE3.7 (AOUT2)
- new net AOUT2_D4: J4.2 (Pin_2), UDRIVE4.6 (AOUT2), UDRIVE4.7 (AOUT2)
- new net AOUT2_L1: J17.2 (Pin_2), ULIFT1.6 (AOUT2), ULIFT1.7 (AOUT2)
- new net AOUT2_L2: J16.2 (Pin_2), ULIFT2.6 (AOUT2), ULIFT2.7 (AOUT2)
- new net AOUT2_L3: J15.2 (Pin_2), ULIFT3.6 (AOUT2), ULIFT3.7 (AOUT2)
- new net AOUT2_L4: J14.2 (Pin_2), ULIFT4.6 (AOUT2), ULIFT4.7 (AOUT2)
- new net AOUT2_T1: J1.2 (Pin_2), UTURN1.6 (AOUT2), UTURN1.7 (AOUT2)
- new net AOUT2_T2: J20.2 (Pin_2), UTURN2.6 (AOUT2), UTURN2.7 (AOUT2)
- new net AOUT2_T3: J13.2 (Pin_2), UTURN3.6 (AOUT2), UTURN3.7 (AOUT2)
- new net AOUT2_T4: J21.2 (Pin_2), UTURN4.6 (AOUT2), UTURN4.7 (AOUT2)
- new net BOUT1_D1: J19.4 (Pin_4), UDRIVE1.10 (BOUT1), UDRIVE1.11 (BOUT1)
- new net BOUT1_D2: J18.4 (Pin_4), UDRIVE2.10 (BOUT1), UDRIVE2.11 (BOUT1)
- new net BOUT1_D3: J2.4 (Pin_4), UDRIVE3.10 (BOUT1), UDRIVE3.11 (BOUT1)
- new net BOUT1_D4: J4.4 (Pin_4), UDRIVE4.10 (BOUT1), UDRIVE4.11 (BOUT1)
- new net BOUT1_L1: J17.4 (Pin_4), ULIFT1.10 (BOUT1), ULIFT1.11 (BOUT1)
- new net BOUT1_L2: J16.4 (Pin_4), ULIFT2.10 (BOUT1), ULIFT2.11 (BOUT1)
- new net BOUT1_L3: J15.4 (Pin_4), ULIFT3.10 (BOUT1), ULIFT3.11 (BOUT1)
- new net BOUT1_L4: J14.4 (Pin_4), ULIFT4.10 (BOUT1), ULIFT4.11 (BOUT1)
- new net BOUT1_T1: J1.4 (Pin_4), UTURN1.10 (BOUT1), UTURN1.11 (BOUT1)
- new net BOUT1_T2: J20.4 (Pin_4), UTURN2.10 (BOUT1), UTURN2.11 (BOUT1)
- new net BOUT1_T3: J13.4 (Pin_4), UTURN3.10 (BOUT1), UTURN3.11 (BOUT1)
- new net BOUT1_T4: J21.4 (Pin_4), UTURN4.10 (BOUT1), UTURN4.11 (BOUT1)
- new net BOUT2_D1: J19.3 (Pin_3), UDRIVE1.8 (BOUT2), UDRIVE1.9 (BOUT2)
- new net BOUT2_D2: J18.3 (Pin_3), UDRIVE2.8 (BOUT2), UDRIVE2.9 (BOUT2)
- new net BOUT2_D3: J2.3 (Pin_3), UDRIVE3.8 (BOUT2), UDRIVE3.9 (BOUT2)
- new net BOUT2_D4: J4.3 (Pin_3), UDRIVE4.8 (BOUT2), UDRIVE4.9 (BOUT2)
- new net BOUT2_L1: J17.3 (Pin_3), ULIFT1.8 (BOUT2), ULIFT1.9 (BOUT2)
- new net BOUT2_L2: J16.3 (Pin_3), ULIFT2.8 (BOUT2), ULIFT2.9 (BOUT2)
- new net BOUT2_L3: J15.3 (Pin_3), ULIFT3.8 (BOUT2), ULIFT3.9 (BOUT2)
- new net BOUT2_L4: J14.3 (Pin_3), ULIFT4.8 (BOUT2), ULIFT4.9 (BOUT2)
- new net BOUT2_T1: J1.3 (Pin_3), UTURN1.8 (BOUT2), UTURN1.9 (BOUT2)
- new net BOUT2_T2: J20.3 (Pin_3), UTURN2.8 (BOUT2), UTURN2.9 (BOUT2)
- new net BOUT2_T3: J13.3 (Pin_3), UTURN3.8 (BOUT2), UTURN3.9 (BOUT2)
- new net BOUT2_T4: J21.3 (Pin_3), UTURN4.8 (BOUT2), UTURN4.9 (BOUT2)
- new net GNDD: JBUCK5_LOGIC1.1 (Pin_1)
- no-connect marks 0 -> 4
Other:
- moved on the sheet: C21, C22, C23, C24, C25, C26, C27, C28, C29, C30, C51, C52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
