File: KiCad/12_Driver_Board/2ESP_Breakout.kicad_sch (KiCad schematic)
At the start: 86 parts, among them J10 Conn_01x02_Socket, J11 Conn_01x02_Socket, J12 Conn_01x02_Socket, J5 Conn_01x02_Socket, J6 Conn_01x02_Socket, J7 Conn_01x02_Socket, J8 Conn_01x02_Socket, J9 Conn_01x02_Socket, U10 PC817, U11 6N137, U12 PC817, U13 PC817, U14 6N137, U15 6N137, U16 PC817, U17 6N137, U18 6N137, U19 PC817, U2 6N137, U20 6N137, U21 PC817, U3 PC817, U4 6N137, U5 PC817, U6 PC817, U7 6N137, U8 PC817, U9 6N137

Commit message: Adding Cad files
Parts:
- C61: renamed from C12; footprint Capacitor_SMD:C_0603_1608Metric -> Capacitor_SMD:C_0805_2012Metric
- C62: renamed from C13; footprint Capacitor_SMD:C_0603_1608Metric -> Capacitor_SMD:C_0805_2012Metric
- C63: renamed from C14; footprint Capacitor_SMD:C_0603_1608Metric -> Capacitor_SMD:C_0805_2012Metric
- C64: renamed from C15; footprint Capacitor_SMD:C_0603_1608Metric -> Capacitor_SMD:C_0805_2012Metric
- C65: renamed from C7; footprint Capacitor_SMD:C_0603_1608Metric -> Capacitor_SMD:C_0805_2012Metric
- C66: renamed from C8; footprint Capacitor_SMD:C_0603_1608Metric -> Capacitor_SMD:C_0805_2012Metric
- C67: renamed from C11; footprint Capacitor_SMD:C_0603_1608Metric -> Capacitor_SMD:C_0805_2012Metric
- C68: renamed from C16; footprint Capacitor_SMD:C_0603_1608Metric -> Capacitor_SMD:C_0805_2012Metric
- C69: renamed from C9; footprint Capacitor_SMD:C_0603_1608Metric -> Capacitor_SMD:C_0805_2012Metric
- C70: renamed from C10; footprint Capacitor_SMD:C_0603_1608Metric -> Capacitor_SMD:C_0805_2012Metric
- R38: renamed from R27; footprint Resistor_SMD:R_0603_1608Metric -> Resistor_SMD:R_0805_2012Metric
- R39: renamed from R26; footprint Resistor_SMD:R_0603_1608Metric -> Resistor_SMD:R_0805_2012Metric
- R40: renamed from R29; footprint Resistor_SMD:R_0603_1608Metric -> Resistor_SMD:R_0805_2012Metric
- R41: renamed from R28; footprint Resistor_SMD:R_0603_1608Metric -> Resistor_SMD:R_0805_2012Metric
- R42: renamed from R31; footprint Resistor_SMD:R_0603_1608Metric -> Resistor_SMD:R_0805_2012Metric
- R43: renamed from R30; footprint Resistor_SMD:R_0603_1608Metric -> Resistor_SMD:R_0805_2012Metric
- R44: renamed from R33; footprint Resistor_SMD:R_0603_1608Metric -> Resistor_SMD:R_0805_2012Metric
- R45: renamed from R34; footprint Resistor_SMD:R_0603_1608Metric -> Resistor_SMD:R_0805_2012Metric
- R46: renamed from R32; footprint Resistor_SMD:R_0603_1608Metric -> Resistor_SMD:R_0805_2012Metric
- R47: renamed from R35; footprint Resistor_SMD:R_0603_1608Metric -> Resistor_SMD:R_0805_2012Metric
- R48: renamed from R36; footprint Resistor_SMD:R_0603_1608Metric -> Resistor_SMD:R_0805_2012Metric
- R49: renamed from R37; footprint Resistor_SMD:R_0603_1608Metric -> Resistor_SMD:R_0805_2012Metric
- R50: renamed from R38; footprint Resistor_SMD:R_0603_1608Metric -> Resistor_SMD:R_0805_2012Metric
- R51: renamed from R39; footprint Resistor_SMD:R_0603_1608Metric -> Resistor_SMD:R_0805_2012Metric
- R52: renamed from R8; footprint Resistor_SMD:R_0603_1608Metric -> Resistor_SMD:R_0805_2012Metric
- R53: renamed from R7; footprint Resistor_SMD:R_0603_1608Metric -> Resistor_SMD:R_0805_2012Metric
- R54: renamed from R6; footprint Resistor_SMD:R_0603_1608Metric -> Resistor_SMD:R_0805_2012Metric
- R55: renamed from R9; footprint Resistor_SMD:R_0603_1608Metric -> Resistor_SMD:R_0805_2012Metric
- R56: renamed from R11; footprint Resistor_SMD:R_0603_1608Metric -> Resistor_SMD:R_0805_2012Metric
- R57: renamed from R4; footprint Resistor_SMD:R_0603_1608Metric -> Resistor_SMD:R_0805_2012Metric
- R58: renamed from R10; footprint Resistor_SMD:R_0603_1608Metric -> Resistor_SMD:R_0805_2012Metric
- R59: renamed from R5; footprint Resistor_SMD:R_0603_1608Metric -> Resistor_SMD:R_0805_2012Metric
- R60: renamed from R13; footprint Resistor_SMD:R_0603_1608Metric -> Resistor_SMD:R_0805_2012Metric
- R61: renamed from R12; footprint Resistor_SMD:R_0603_1608Metric -> Resistor_SMD:R_0805_2012Metric
- R62: renamed from R23; footprint Resistor_SMD:R_0603_1608Metric -> Resistor_SMD:R_0805_2012Metric
- R63: renamed from R22; footprint Resistor_SMD:R_0603_1608Metric -> Resistor_SMD:R_0805_2012Metric
- R64: renamed from R43; footprint Resistor_SMD:R_0603_1608Metric -> Resistor_SMD:R_0805_2012Metric
- R65: renamed from R40; footprint Resistor_SMD:R_0603_1608Metric -> Resistor_SMD:R_0805_2012Metric
- R66: renamed from R42; footprint Resistor_SMD:R_0603_1608Metric -> Resistor_SMD:R_0805_2012Metric
- R67: renamed from R41; footprint Resistor_SMD:R_0603_1608Metric -> Resistor_SMD:R_0805_2012Metric
- R68: renamed from R20; footprint Resistor_SMD:R_0603_1608Metric -> Resistor_SMD:R_0805_2012Metric
- R69: renamed from R14; footprint Resistor_SMD:R_0603_1608Metric -> Resistor_SMD:R_0805_2012Metric
- R70: renamed from R18; footprint Resistor_SMD:R_0603_1608Metric -> Resistor_SMD:R_0805_2012Metric
- R71: renamed from R15; footprint Resistor_SMD:R_0603_1608Metric -> Resistor_SMD:R_0805_2012Metric
- R72: renamed from R21; footprint Resistor_SMD:R_0603_1608Metric -> Resistor_SMD:R_0805_2012Metric
- R73: renamed from R16; footprint Resistor_SMD:R_0603_1608Metric -> Resistor_SMD:R_0805_2012Metric
- R74: renamed from R19; footprint Resistor_SMD:R_0603_1608Metric -> Resistor_SMD:R_0805_2012Metric
- R75: renamed from R17; footprint Resistor_SMD:R_0603_1608Metric -> Resistor_SMD:R_0805_2012Metric
- R76: renamed from R25; footprint Resistor_SMD:R_0603_1608Metric -> Resistor_SMD:R_0805_2012Metric
- R77: renamed from R24; footprint Resistor_SMD:R_0603_1608Metric -> Resistor_SMD:R_0805_2012Metric
- renumbered ESP3L_2 to ESP3L_1, ESP3L_1 to ESP3L_2, ESP3L_3 to ESP3R_2
Connections:
- net +5V: no longer ESP1L_1.15 (VIN), ESP2L_1.15 (VIN), ESP3L_1.15 (VIN), ESP3L_2.15 (VIN)
- net GND: no longer ESP1L_1.14 (GND), ESP1R_1.14 (GND), ESP2L_1.14 (GND), ESP2R_1.14 (GND), ESP3L_1.14 (GND), ESP3L_2.14 (GND), ESP3R_1.14 (GND), ESP3R_2.14 (GND), J10.2 (Pin_2), J11.2 (Pin_2), J12.2 (Pin_2), J5.2 (Pin_2), J6.2 (Pin_2), J7.2 (Pin_2), J8.2 (Pin_2), J9.2 (Pin_2), R38.1, R40.1, R42.1, R44.1, R46.1, R48.1, R50.1, R52.1, R54.1, R56.1, R58.1, R60.1, R62.1, R64.1, R66.1, R68.1, R70.1, R72.1, R74.1, R76.1
- new net +5VD: ESP1L_1.15 (VIN), ESP2L_1.15 (VIN), ESP3L_1.15 (VIN), ESP3L_2.15 (VIN)
- new net GNDD: ESP1L_1.14 (GND), ESP1R_1.14 (GND), ESP2L_1.14 (GND), ESP2R_1.14 (GND), ESP3L_1.14 (GND), ESP3L_2.14 (GND), ESP3R_1.14 (GND), ESP3R_2.14 (GND), J10.2 (Pin_2), J11.2 (Pin_2), J12.2 (Pin_2), J5.2 (Pin_2), J6.2 (Pin_2), J7.2 (Pin_2), J8.2 (Pin_2), J9.2 (Pin_2), R38.1, R40.1, R42.1, R44.1, R46.1, R48.1, R50.1, R52.1, R54.1, R56.1, R58.1, R60.1, R62.1, R64.1, R66.1, R68.1, R70.1, R72.1, R74.1, R76.1
